File: Matriz_Led.sch (KiCad schematic (older format))
At the start: 22 parts, among them Q1 2N3904BU, Q2 2N3904BU, Q3 2N3904BU, Q4 2N3904BU, Q5 2N3904BU, U1 74HC595, U2 74HC595, U3 Matriz_5x7

Commit message: añaadido zocalo para sensor de temperatura y primera distribucion sobre la PCB
Parts:
- removed Q1, Q2, Q3, Q4, Q5: 2N3904BU, Transistors:TO-92_EnLinea_Estrecho_Oval, symbol Q_NPN_EBC
- added Q1, Q2, Q3, Q4, Q5: SMBT3904, TO_SOT_Packages_SMD:SOT-23, symbol BC849
- C1, C2: footprint Capacitors_ThroughHole:C_Disc_D3_P2.5 -> Capacitors_SMD:C_0805
- R1, R10, R11, R12, R2, R3, R4, R5, R6, R7, R8, R9: footprint Resistencias:Resistencia_1_4_W_10_mm -> Resistors_SMD:R_0805

Commit message: añadiendo valores del distribuidor a los componentes
Parts:
- C1, C2: Fabricante (none) -> SAMSUNG; Provedor (none) -> TME; Ref (none) -> CL21B104KBCNNNC; Ref_Proveedor (none) -> CL21B104KBCNNNC
- R1, R10, R11, R12, R5: Fabricante SR_PASSIVES -> VISHAY; Potencia 1/4W -> 1/8W; Ref CF1/4W-1K -> CRCW08051K00FKEA; Ref_Proveedor CF1/4W-1K -> CRCW08051K00FKEA; Tolerancia 5% -> 1%
- R2, R3, R4, R6, R7, R8, R9: Fabricante SR_PASSIVES -> VISHAY; Potencia 1/4W -> 1/8W; Ref CF1/4W-120R -> CRCW0805120RFKTABC; Ref_Proveedor CF1/4W-120R -> CRCW0805120RFKTABC; Tolerancia 5% -> 1%

Commit message: ordenar referencias de componentes
Parts:
- renumbered C1 to C3, C2 to C4, R6 to R1, R7 to R3, R3 to R4, R8 to R5, R4 to R6, R9 to R7, R1 to R8, R5 to R9, U1 to U4, U2 to U5
Changed lines of the file:
@@
 $Descr A4 11693 8268
 encoding utf-8
-Sheet 2 15
+Sheet 4 15
 Title ""
 Date ""
@@
 $EndComp
 $Comp
-L GND #PWR057
+L GND #PWR14
 U 1 1 5793BD55
 P 5700 6100
-F 0 "#PWR057" H 5700 5850 50  0001 C CNN
+F 0 "#PWR14" H 5700 5850 50  0001 C CNN
 F 1 "GND" H 5700 5950 50  0000 C CNN
 F 2 "" H 5700 6100 50  0000 C CNN
@@
 $EndComp
 $Comp
-L R R6
+L R R1
 U 1 1 5793BD61
 P 4900 2000
-F 0 "R6" V 4980 2000 50  0000 C CNN
+F 0 "R1" V 4980 2000 50  0000 C CNN
 F 1 "120" V 4900 2000 50  0000 C CNN
 F 2 "Resistors_SMD:R_0805" V 4830 2000 50  0001 C CNN
@@
 $EndComp
 $Comp
-L 74HC595 U1
+L 74HC595 U4
 U 1 1 5793BDAF
 P 3300 2450
-F 0 "U1" H 3450 3050 50  0000 C CNN
+F 0 "U4" H 3450 3050 50  0000 C CNN
 F 1 "74HC595" H 3300 1850 50  0000 C CNN
 F 2 "Housings_SOIC:SOIC-16_3.9x9.9mm_Pitch1.27mm" H 3300 2450 50  0001 C CNN
@@
 $EndComp
 $Comp
-L GND #PWR058
+L GND #PWR13
 U 1 1 5793BDB6
 P 2350 4700
-F 0 "#PWR058" H 2350 4450 50  0001 C CNN
+F 0 "#PWR13" H 2350 4450 50  0001 C CNN
 F 1 "GND" H 2350 4550 50  0000 C CNN
 F 2 "" H 2350 4700 50  0000 C CNN
@@
 $EndComp
 $Comp
-L C C1
+L C C3
 U 1 1 5793BDC2
 P 1150 2350
-F 0 "C1" H 1175 2450 50  0000 L CNN
+F 0 "C3" H 1175 2450 50  0000 L CNN
 F 1 "100n" H 1175 2250 50  0000 L CNN
 F 2 "Capacitors_SMD:C_0805" H 1188 2200 50  0001 C CNN
@@
 $EndComp
 $Comp
-L +5V #PWR059
+L +5V #PWR12
 U 1 1 5793BDC9
 P 2150 1850
-F 0 "#PWR059" H 2150 1700 50  0001 C CNN
+F 0 "#PWR12" H 2150 1700 50  0001 C CNN
 F 1 "+5V" H 2150 1990 50  0000 C CNN
 F 2 "" H 2150 1850 50  0000 C CNN
@@
 $EndComp
 $Comp
-L GND #PWR060
+L GND #PWR9
 U 1 1 5793BDCF
 P 1150 2600
-F 0 "#PWR060" H 1150 2350 50  0001 C CNN
+F 0 "#PWR9" H 1150 2350 50  0001 C CNN
 F 1 "GND" H 1150 2450 50  0000 C CNN
 F 2 "" H 1150 2600 50  0000 C CNN
@@
 $EndComp
 $Comp
-L +5V #PWR061
+L +5V #PWR8
 U 1 1 5793BDD5
 P 1150 2050
-F 0 "#PWR061" H 1150 1900 50  0001 C CNN
+F 0 "#PWR8" H 1150 1900 50  0001 C CNN
 F 1 "+5V" H 1150 2190 50  0000 C CNN
 F 2 "" H 1150 2050 50  0000 C CNN
@@
 $EndComp
 $Comp
-L R R3
+L R R4
 U 1 1 5793BE24
 P 4550 2300
-F 0 "R3" V 4630 2300 50  0000 C CNN
+F 0 "R4" V 4630 2300 50  0000 C CNN
 F 1 "120" V 4550 2300 50  0000 C CNN
 F 2 "Resistors_SMD:R_0805" V 4480 2300 50  0001 C CNN
@@
 $EndComp
 $Comp
-L R R4
+L R R6
 U 1 1 5793BE31
 P 4550 2500
-F 0 "R4" V 4630 2500 50  0000 C CNN
+F 0 "R6" V 4630 2500 50  0000 C CNN
 F 1 "120" V 4550 2500 50  0000 C CNN
 F 2 "Resistors_SMD:R_0805" V 4480 2500 50  0001 C CNN
@@
 $EndComp
 $Comp
-L R R7
+L R R3
 U 1 1 5793BE3E
 P 4900 2200
-F 0 "R7" V 4980 2200 50  0000 C CNN
+F 0 "R3" V 4980 2200 50  0000 C CNN
 F 1 "120" V 4900 2200 50  0000 C CNN
 F 2 "Resistors_SMD:R_0805" V 4830 2200 50  0001 C CNN
@@
 $EndComp
 $Comp
-L R R8
+L R R5
 U 1 1 5793BE4B
 P 4900 2400
-F 0 "R8" V 4980 2400 50  0000 C CNN
+F 0 "R5" V 4980 2400 50  0000 C CNN
 F 1 "120" V 4900 2400 50  0000 C CNN
 F 2 "Resistors_SMD:R_0805" V 4830 2400 50  0001 C CNN
@@
 $EndComp
 $Comp
-L R R9
+L R R7
 U 1 1 5793BE58
 P 4900 2600
-F 0 "R9" V 4980 2600 50  0000 C CNN
+F 0 "R7" V 4980 2600 50  0000 C CNN
 F 1 "120" V 4900 2600 50  0000 C CNN
 F 2 "Resistors_SMD:R_0805" V 4830 2600 50  0001 C CNN
@@
 $EndComp
 $Comp
-L R R1
+L R R8
 U 1 1 5793BE65
 P 4300 3800
-F 0 "R1" V 4200 3800 50  0000 C CNN
+F 0 "R8" V 4200 3800 50  0000 C CNN
 F 1 "1K" V 4300 3800 50  0000 C CNN
 F 2 "Resistors_SMD:R_0805" V 4230 3800 50  0001 C CNN
@@
 $EndComp
 $Comp
-L R R5
+L R R9
 U 1 1 5793BE72
 P 4700 4200
-F 0 "R5" V 4600 4200 50  0000 C CNN
+F 0 "R9" V 4600 4200 50  0000 C CNN
 F 1 "1K" V 4700 4200 50  0000 C CNN
 F 2 "Resistors_SMD:R_0805" V 4630 4200 50  0001 C CNN
@@
 MATRIZ DE LEDS 5x7
 $Comp
-L 74HC595 U2
+L 74HC595 U5
 U 1 1 5793BEAB
 P 3300 4250
-F 0 "U2" H 3450 4850 50  0000 C CNN
+F 0 "U5" H 3450 4850 50  0000 C CNN
 F 1 "74HC595" H 3300 3650 50  0000 C CNN
 F 2 "Housings_SOIC:SOIC-16_3.9x9.9mm_Pitch1.27mm" H 3300 4250 50  0001 C CNN
@@
 NoConn ~ 4000 4700
 $Comp
-L C C2
+L C C4
 U 1 1 5793BED8
 P 1150 4150
-F 0 "C2" H 1175 4250 50  0000 L CNN
+F 0 "C4" H 1175 4250 50  0000 L CNN
 F 1 "100n" H 1175 4050 50  0000 L CNN
 F 2 "Capacitors_SMD:C_0805" H 1188 4000 50  0001 C CNN
@@
 $EndComp
 $Comp
-L GND #PWR062
+L GND #PWR11
 U 1 1 5793BEDF
 P 1150 4400
-F 0 "#PWR062" H 1150 4150 50  0001 C CNN
+F 0 "#PWR11" H 1150 4150 50  0001 C CNN
 F 1 "GND" H 1150 4250 50  0000 C CNN
 F 2 "" H 1150 4400 50  0000 C CNN
@@
 $EndComp
 $Comp
-L +5V #PWR063
+L +5V #PWR10
 U 1 1 5793BEE5
 P 1150 3850
-F 0 "#PWR063" H 1150 3700 50  0001 C CNN
+F 0 "#PWR10" H 1150 3700 50  0001 C CNN
 F 1 "+5V" H 1150 3990 50  0000 C CNN
 F 2 "" H 1150 3850 50  0000 C CNN
@@
 30 0C C3 30 0C C3 30 0C C3 30 3E 7B 4C E0 30 0C C3 30 0C C3 30 0C C3 30 0C E3 B3 C7 04 0E C3 30
 0C C3 30 0C C3 30 0C C3 30 3E 7B 4C E0 30 0C C3 30 0C C3 30 0C C3 30 0C E3 B3 E7 DF 01 18 4D 27
-06 D5 63 A7 50 00 00 00 00 49 45 4E 44 AE 42 60 82 FF
+06 D5 63 A7 50 00 00 00 00 49 45 4E 44 AE 42 60 82 00
 EndData
 $EndBitmap

Commit message: Actualizado el esquema electrico
Other:
- moved on the sheet: C3, C4, Q1, Q2, Q3, Q4, Q5, R1, R10, R11, R12, R2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
