File: Control.sch (KiCad schematic (older format))
At the start: 1 part, among them U5 Arduino_Nano

Commit message: añaadido zocalo para sensor de temperatura y primera distribucion sobre la PCB
Connections:
- no-connect marks 3 -> 4
Other:
- note added: "Bluetooth Tx\n\nBluetooth Rx\n\nD2\n\nBuzzer\n\nReloj de carga de salidas del registro despl.\n\nServo nº 1\n\nServo nº 2\n\nUltrasonidos Trigg\n\nUltrasonidos Echo\n\nLed RGB Rojo\n\nLed RGB Verde\n\nLed RGB Azul\n\nDato de entrada al registro de despl.\n\nReloj de carga serie del registro despl.\n\nPulsadores - Bit 0\n\nPulsadores - Bit 1\n\nBluetooth - Key\n\nSensor DTH Dato\n\nI2C - SDA\n\nI2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"
- note removed: "Bluetooth Tx\n\nBluetooth Rx\n\nD2\n\nBuzzer\n\nReloj de carga de salidas del registro despl.\n\nServo nº 1\n\nServo nº 2\n\nUltrasonidos Trigg\n\nUltrasonidos Echo\n\nLed RGB Rojo\n\nLed RGB Verde\n\nLed RGB Azul\n\nDato de entrada al registro de despl.\n\nReloj de carga serie del registro despl.\n\nPulsadores - Bit 0\n\nPulsadores - Bit 1\n\nBluetooth - Key\n\nA3\n\nI2C - SDA\n\nI2C - SCL\n\nLD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"
Changed lines of the file:
@@
 $Descr A4 11693 8268
 encoding utf-8
-Sheet 4 13
+Sheet 4 14
 Title ""
 Date ""
@@
 Text GLabel 7650 3750 2    60   Input ~ 0
 A4
-Text GLabel 7650 3900 2    60   Input ~ 0
+Text GLabel 7650 3900 2    60   BiDi ~ 0
 A3
 Text GLabel 7650 4050 2    60   Input ~ 0
@@
 D0\n\nD1\n\nD2\n\nD3\n\nD4\n\nD5\n\nD6\n\nD7\n\nD8\n\nD9\n\nD10\n\nD11\n\nD12\n\nD13\n\nA0\n\nA1\n\nA2\n\nA3\n\nA4\n\nA5\n\nA6\n\nA7
 Text Notes 1250 6900 0    79   ~ 0
-Bluetooth Tx\n\nBluetooth Rx\n\nD2\n\nBuzzer\n\nReloj de carga de salidas del registro despl.\n\nServo nº 1\n\nServo nº 2\n\nUltrasonidos Trigg\n\nUltrasonidos Echo\n\nLed RGB Rojo\n\nLed RGB Verde\n\nLed RGB Azul\n\nDato de entrada al registro de despl.\n\nReloj de carga serie del registro despl.\n\nPulsadores - Bit 0\n\nPulsadores - Bit 1\n\nBluetooth - Key\n\nA3\n\nI2C - SDA\n\nI2C - SCL\n\nLDR\n\nPotenciometro
+Bluetooth Tx\n\nBluetooth Rx\n\nD2\n\nBuzzer\n\nReloj de carga de salidas del registro despl.\n\nServo nº 1\n\nServo nº 2\n\nUltrasonidos Trigg\n\nUltrasonidos Echo\n\nLed RGB Rojo\n\nLed RGB Verde\n\nLed RGB Azul\n\nDato de entrada al registro de despl.\n\nReloj de carga serie del registro despl.\n\nPulsadores - Bit 0\n\nPulsadores - Bit 1\n\nBluetooth - Key\n\nSensor DTH Dato\n\nI2C - SDA\n\nI2C - SCL\n\nLDR\n\nPotenciometro
 Wire Notes Line
 	800  1050 800  7000
@@
 	1    0    0    -1
 $EndComp
+NoConn ~ 5750 3650
 $EndSCHEMATC

Commit message: finalizado enrutado provisional
Connections:
- no-connect marks 4 -> 3
Other:
- note added: "Bluetooth Tx\n\nBluetooth Rx\n\nEncoder canal A\n\nBuzzer\n\nReloj de carga de salidas del registro despl.\n\nServo nº 1\n\nServo nº 2\n\nUltrasonidos Echo\n\nUltrasonidos Trigg\n\nLed RGB Rojo\n\nLed RGB Verde\n\nLed RGB Azul\n\nDato de entrada al registro de despl.\n\nReloj de carga serie del registro despl.\n\nPulsadores - Bit 0\n\nPulsadores - Bit 1\n\nEncoder canal B\n\nSensor DTH Dato\n\nI2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"
- note removed: "Bluetooth Tx\n\nBluetooth Rx\n\nD2\n\nBuzzer\n\nReloj de carga de salidas del registro despl.\n\nServo nº 1\n\nServo nº 2\n\nUltrasonidos Trigg\n\nUltrasonidos Echo\n\nLed RGB Rojo\n\nLed RGB Verde\n\nLed RGB Azul\n\nDato de entrada al registro de despl.\n\nReloj de carga serie del registro despl.\n\nPulsadores - Bit 0\n\nPulsadores - Bit 1\n\nBluetooth - Key\n\nSensor DTH Dato\n\nI2C - SDA\n\nI2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"
Changed lines of the file:
@@
 $Descr A4 11693 8268
 encoding utf-8
-Sheet 4 14
+Sheet 3 15
 Title ""
 Date ""
@@
 NoConn ~ 7100 3000
 $Comp
-L GND #PWR013
+L GND #PWR06
 U 1 1 5793CBBD
 P 5550 5300
-F 0 "#PWR013" H 5550 5050 50  0001 C CNN
+F 0 "#PWR06" H 5550 5050 50  0001 C CNN
 F 1 "GND" H 5550 5150 50  0000 C CNN
 F 2 "" H 5550 5300 50  0000 C CNN
@@
 $EndComp
 $Comp
-L GND #PWR014
+L GND #PWR07
 U 1 1 5793CBC3
 P 7200 5300
-F 0 "#PWR014" H 7200 5050 50  0001 C CNN
+F 0 "#PWR07" H 7200 5050 50  0001 C CNN
 F 1 "GND" H 7200 5150 50  0000 C CNN
 F 2 "" H 7200 5300 50  0000 C CNN
@@
 	5800 3300 5250 3300
 $Comp
-L +5V #PWR015
+L +5V #PWR08
 U 1 1 5793CBF2
 P 7300 2150
-F 0 "#PWR015" H 7300 2000 50  0001 C CNN
+F 0 "#PWR08" H 7300 2000 50  0001 C CNN
 F 1 "+5V" H 7300 2290 50  0000 C CNN
 F 2 "" H 7300 2150 50  0000 C CNN
@@
 D0\n\nD1\n\nD2\n\nD3\n\nD4\n\nD5\n\nD6\n\nD7\n\nD8\n\nD9\n\nD10\n\nD11\n\nD12\n\nD13\n\nA0\n\nA1\n\nA2\n\nA3\n\nA4\n\nA5\n\nA6\n\nA7
 Text Notes 1250 6900 0    79   ~ 0
-Bluetooth Tx\n\nBluetooth Rx\n\nD2\n\nBuzzer\n\nReloj de carga de salidas del registro despl.\n\nServo nº 1\n\nServo nº 2\n\nUltrasonidos Trigg\n\nUltrasonidos Echo\n\nLed RGB Rojo\n\nLed RGB Verde\n\nLed RGB Azul\n\nDato de entrada al registro de despl.\n\nReloj de carga serie del registro despl.\n\nPulsadores - Bit 0\n\nPulsadores - Bit 1\n\nBluetooth - Key\n\nSensor DTH Dato\n\nI2C - SDA\n\nI2C - SCL\n\nLDR\n\nPotenciometro
+Bluetooth Tx\n\nBluetooth Rx\n\nEncoder canal A\n\nBuzzer\n\nReloj de carga de salidas del registro despl.\n\nServo nº 1\n\nServo nº 2\n\nUltrasonidos Echo\n\nUltrasonidos Trigg\n\nLed RGB Rojo\n\nLed RGB Verde\n\nLed RGB Azul\n\nDato de entrada al registro de despl.\n\nReloj de carga serie del registro despl.\n\nPulsadores - Bit 0\n\nPulsadores - Bit 1\n\nEncoder canal B\n\nSensor DTH Dato\n\nI2C - SDA\n\nI2C - SCL\n\nLDR\n\nPotenciometro
 Wire Notes Line
 	800  1050 800  7000
@@
 	4050 1050 800  1050
 $Comp
-L +3V3 #PWR016
+L +3V3 #PWR09
 U 1 1 57954065
 P 7450 2400
-F 0 "#PWR016" H 7450 2250 50  0001 C CNN
+F 0 "#PWR09" H 7450 2250 50  0001 C CNN
 F 1 "+3V3" H 7465 2573 50  0000 C CNN
 F 2 "" H 7450 2400 50  0000 C CNN
@@
 	1    0    0    -1
 $EndComp
-NoConn ~ 5750 3650
 $EndSCHEMATC

Commit message: ordenar referencias de componentes
Parts:
- renumbered U5 to U1
Changed lines of the file:
@@
 $Descr A4 11693 8268
 encoding utf-8
-Sheet 3 15
+Sheet 2 15
 Title ""
 Date ""
@@
 $EndDescr
 $Comp
-L Arduino_Nano U5
+L Arduino_Nano U1
 U 1 1 5793CBB2
 P 6450 4950
-F 0 "U5" H 6100 4800 60  0000 C CNN
+F 0 "U1" H 6100 4800 60  0000 C CNN
 F 1 "Arduino_Nano" H 6500 7450 60  0000 C CNN
 F 2 "Arduino:Arduino_Nano" H 6450 4950 60  0001 C CNN
@@
 NoConn ~ 7100 3000
 $Comp
-L GND #PWR06
+L GND #PWR1
 U 1 1 5793CBBD
 P 5550 5300
-F 0 "#PWR06" H 5550 5050 50  0001 C CNN
+F 0 "#PWR1" H 5550 5050 50  0001 C CNN
 F 1 "GND" H 5550 5150 50  0000 C CNN
 F 2 "" H 5550 5300 50  0000 C CNN
@@
 $EndComp
 $Comp
-L GND #PWR07
+L GND #PWR2
 U 1 1 5793CBC3
 P 7200 5300
-F 0 "#PWR07" H 7200 5050 50  0001 C CNN
+F 0 "#PWR2" H 7200 5050 50  0001 C CNN
 F 1 "GND" H 7200 5150 50  0000 C CNN
 F 2 "" H 7200 5300 50  0000 C CNN
@@
 	5800 3300 5250 3300
 $Comp
-L +5V #PWR08
+L +5V #PWR3
 U 1 1 5793CBF2
 P 7300 2150
-F 0 "#PWR08" H 7300 2000 50  0001 C CNN
+F 0 "#PWR3" H 7300 2000 50  0001 C CNN
 F 1 "+5V" H 7300 2290 50  0000 C CNN
 F 2 "" H 7300 2150 50  0000 C CNN
@@
 08 82 20 08 6E 93 D0 F8 20 08 82 20 B8 4D 42 E3 83 20 08 82 E0 36 09 8D 0F 82 20 08 82 DB 24 34
 3E 08 82 20 08 6E 93 D0 F8 20 08 82 20 B8 4D 42 E3 83 20 08 82 E0 36 09 8D 0F 82 20 08 82 DB E4
-FF 01 8A 98 D1 7C B7 EF D0 30 00 00 00 00 49 45 4E 44 AE 42 60 82 00
+FF 01 8A 98 D1 7C B7 EF D0 30 00 00 00 00 49 45 4E 44 AE 42 60 82 BD
 EndData
 $EndBitmap
@@
 	4050 1050 800  1050
 $Comp
-L +3V3 #PWR09
+L +3V3 #PWR4
 U 1 1 57954065
 P 7450 2400
-F 0 "#PWR09" H 7450 2250 50  0001 C CNN
+F 0 "#PWR4" H 7450 2250 50  0001 C CNN
 F 1 "+3V3" H 7465 2573 50  0000 C CNN
 F 2 "" H 7450 2400 50  0000 C CNN
