File: Control.sch (KiCad schematic (older format))
At the start: 1 part, among them U1 Arduino_Nano

Commit message: añadidos driver para led y conectores para fotodiodos infrarrojos
Connections:
- net D0: no longer names the net of U1.2 (RX0)
- net D1: no longer names the net of U1.1 (TX1)
- no-connect marks 3 -> 5
Other:
- note added: "USB Tx\n\nUSB Rx\n\nEncoder canal A\n\nInterrupción Acelerómetro\n\nReloj de carga de salidas del registro despl.\n\nEncoder canal B\n\nInfrarrojos Izquierdo\n\nUltrasonidos Echo\n\nUltrasonidos Trigg\n\nInfrarrojos Derecho\n\nInalámbrico Tx\n\nInalámbrico Rx\n\nDato de entrada al registro de despl.\n\nReloj de carga serie del registro despl.\n\nPulsadores - Bit 0\n\nPulsadores - Bit 1\n\nPulsado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"
- note removed: "Bluetooth Tx\n\nBluetooth Rx\n\nEncoder canal A\n\nBuzzer\n\nReloj de carga de salidas del registro despl.\n\nServo nº 1\n\nServo nº 2\n\nUltrasonidos Echo\n\nUltrasonidos Trigg\n\nLed RGB Rojo\n\nLed RGB Verde\n\nLed RGB Azul\n\nDato de entrada al registro de despl.\n\nReloj de carga serie del registro despl.\n\nPulsadores - Bit 0\n\nPulsadores - Bit 1\n\nEncoder canal B\n\nSensor DTH Dato\n\nI2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"
Changed lines of the file:
@@
 EESchema Schematic File Version 2
+LIBS:Interfaces
+LIBS:Nano_PB-rescue
 LIBS:Sensores
 LIBS:power
@@
 LIBS:valves
 LIBS:MyLibrary
+LIBS:matriz_led
 LIBS:Nano_PB-cache
-EELAYER 25 0
+EELAYER 26 0
 EELAYER END
 $Descr A4 11693 8268
 encoding utf-8
-Sheet 2 15
+Sheet 2 16
 Title "Control de la placa"
-Date "2016-08-07"
-Rev "V.0.2"
+Date "2017-01-04"
+Rev "V.0.3"
 Comp "NanoPlayBoard"
 Comment1 "Creada por Antonio Morales"
@@
 Text GLabel 7650 4800 2    60   Output ~ 0
 D13
-Text GLabel 5250 2700 0    60   Input ~ 0
-D1
-Wire Wire Line
-	5250 2700 5800 2700
-Wire Wire Line
-	5250 2850 5800 2850
-Text GLabel 5250 2850 0    60   Input ~ 0
-D0
 Text GLabel 5250 3300 0    60   Input ~ 0
 D2
-Text GLabel 5250 3450 0    60   Output ~ 0
+Text GLabel 5250 3450 0    60   Input ~ 0
 D3
 Text GLabel 5250 3600 0    60   Input ~ 0
@@
 08 82 20 08 6E 93 D0 F8 20 08 82 20 B8 4D 42 E3 83 20 08 82 E0 36 09 8D 0F 82 20 08 82 DB 24 34
 3E 08 82 20 08 6E 93 D0 F8 20 08 82 20 B8 4D 42 E3 83 20 08 82 E0 36 09 8D 0F 82 20 08 82 DB E4
-FF 01 8A 98 D1 7C B7 EF D0 30 00 00 00 00 49 45 4E 44 AE 42 60 82 00
+FF 01 8A 98 D1 7C B7 EF D0 30 00 00 00 00 49 45 4E 44 AE 42 60 82
 EndData
 $EndBitmap
@@
 D0\n\nD1\n\nD2\n\nD3\n\nD4\n\nD5\n\nD6\n\nD7\n\nD8\n\nD9\n\nD10\n\nD11\n\nD12\n\nD13\n\nA0\n\nA1\n\nA2\n\nA3\n\nA4\n\nA5\n\nA6\n\nA7
 Text Notes 1250 6900 0    79   ~ 0
-Bluetooth Tx\n\nBluetooth Rx\n\nEncoder canal A\n\nBuzzer\n\nReloj de carga de salidas del registro despl.\n\nServo nº 1\n\nServo nº 2\n\nUltrasonidos Echo\n\nUltrasonidos Trigg\n\nLed RGB Rojo\n\nLed RGB Verde\n\nLed RGB Azul\n\nDato de entrada al registro de despl.\n\nReloj de carga serie del registro despl.\n\nPulsadores - Bit 0\n\nPulsadores - Bit 1\n\nEncoder canal B\n\nSensor DTH Dato\n\nI2C - SDA\n\nI2C - SCL\n\nLDR\n\nPotenciometro
+USB Tx\n\nUSB Rx\n\nEncoder canal A\n\nInterrupción Acelerómetro\n\nReloj de carga de salidas del registro despl.\n\nEncoder canal B\n\nInfrarrojos Izquierdo\n\nUltrasonidos Echo\n\nUltrasonidos Trigg\n\nInfrarrojos Derecho\n\nInalámbrico Tx\n\nInalámbrico Rx\n\nDato de entrada al registro de despl.\n\nReloj de carga serie del registro despl.\n\nPulsadores - Bit 0\n\nPulsadores - Bit 1\n\nPulsadores - Detección Pulsación\n\nSensor DTH Dato\n\nI2C - SDA\n\nI2C - SCL\n\nLDR\n\nPotenciometro
 Wire Notes Line
 	800  1050 800  7000
@@
 50 17 92 01 51 92 64 0C CE 27 7B 4E 87 A3 FC C9 E9 39 BC D0 3B DC 1F CF E6 3C 60 30 83 10 3D 18
 F4 0B 89 52 73 00 8B 80 91 08 28 22 8F 6D AB AA BD D3 E7 C4 3E A7 59 B4 A9 94 4D 1C A1 84 52 AC
-9A 46 F6 7A E1 FF 00 F0 A4 0C 74 26 CB 7B D1 00 00 00 00 49 45 4E 44 AE 42 60 82 00
+9A 46 F6 7A E1 FF 00 F0 A4 0C 74 26 CB 7B D1 00 00 00 00 49 45 4E 44 AE 42 60 82
 EndData
 $EndBitmap
+NoConn ~ 5800 2700
+NoConn ~ 5800 2850
 $EndSCHEMATC

Commit message: Se añade un expansor GPIO al esquema y se elminan registros y codificador
Connections:
- net D13: no longer names the net of U1.16 (D13)
- net D4 renamed ~RESET
- no-connect marks 5 -> 6
Other:
- note added: "USB Tx\n\nUSB Rx\n\nEncoder canal A\n\nInterrupción Acelerómetro\n\nReset Perifericos\n\nEncoder canal B\n\nInfrarrojos Izquierdo\n\nUltrasonidos Echo\n\nUltrasonidos Trigg\n\nInfrarrojos Derecho\n\nInalámbrico Tx\n\nInalámbrico Rx\n\nSensor DTH Dato\n\nLibre\n\nCapacitivo 1\n\nCapacitivo 2\n\nCapacitivo 3\n\nCapacitivo 4\n\nI2C - SDA\n\nI2C - SCL\n\nLDR\n\nPotenciometro"
- note removed: "USB Tx\n\nUSB Rx\n\nEncoder canal A\n\nInterrupción Acelerómetro\n\nReloj de carga de salidas del registro despl.\n\nEncoder canal B\n\nInfrarrojos Izquierdo\n\nUltrasonidos Echo\n\nUltrasonidos Trigg\n\nInfrarrojos Derecho\n\nInalámbrico Tx\n\nInalámbrico Rx\n\nDato de entrada al registro de despl.\n\nReloj de carga serie del registro despl.\n\nPulsadores - Bit 0\n\nPulsadores - Bit 1\n\nPulsado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"
Changed lines of the file:
@@
 LIBS:MyLibrary
 LIBS:matriz_led
+LIBS:Pasivos
 LIBS:Nano_PB-cache
 EELAYER 26 0
@@
 $Descr A4 11693 8268
 encoding utf-8
-Sheet 2 16
+Sheet 2 17
 Title "Control de la placa"
-Date "2017-01-04"
-Rev "V.0.3"
+Date "2017-01-19"
+Rev "V.0.4"
 Comp "NanoPlayBoard"
 Comment1 "Creada por Antonio Morales"
@@
 	7100 4650 7450 4650
 Wire Wire Line
-	7100 4800 7650 4800
-Wire Wire Line
 	5800 4800 5250 4800
 Wire Wire Line
@@
 Text GLabel 7650 3750 2    60   Input ~ 0
 A4
-Text GLabel 7650 3900 2    60   BiDi ~ 0
+Text GLabel 7650 3900 2    60   Input ~ 0
 A3
 Text GLabel 7650 4050 2    60   Input ~ 0
@@
 Text GLabel 7650 4350 2    60   Input ~ 0
 A0
-Text GLabel 7650 4800 2    60   Output ~ 0
-D13
 Text GLabel 5250 3300 0    60   Input ~ 0
 D2
 Text GLabel 5250 3450 0    60   Input ~ 0
 D3
-Text GLabel 5250 3600 0    60   Input ~ 0
-D4
+Text GLabel 5250 3600 0    60   Output ~ 0
+~RESET
 Text GLabel 5250 3750 0    60   Output ~ 0
 D5
@@
 D0\n\nD1\n\nD2\n\nD3\n\nD4\n\nD5\n\nD6\n\nD7\n\nD8\n\nD9\n\nD10\n\nD11\n\nD12\n\nD13\n\nA0\n\nA1\n\nA2\n\nA3\n\nA4\n\nA5\n\nA6\n\nA7
 Text Notes 1250 6900 0    79   ~ 0
-USB Tx\n\nUSB Rx\n\nEncoder canal A\n\nInterrupción Acelerómetro\n\nReloj de carga de salidas del registro despl.\n\nEncoder canal B\n\nInfrarrojos Izquierdo\n\nUltrasonidos Echo\n\nUltrasonidos Trigg\n\nInfrarrojos Derecho\n\nInalámbrico Tx\n\nInalámbrico Rx\n\nDato de entrada al registro de despl.\n\nReloj de carga serie del registro despl.\n\nPulsadores - Bit 0\n\nPulsadores - Bit 1\n\nPulsadores - Detección Pulsación\n\nSensor DTH Dato\n\nI2C - SDA\n\nI2C - SCL\n\nLDR\n\nPotenciometro
+USB Tx\n\nUSB Rx\n\nEncoder canal A\n\nInterrupción Acelerómetro\n\nReset Perifericos\n\nEncoder canal B\n\nInfrarrojos Izquierdo\n\nUltrasonidos Echo\n\nUltrasonidos Trigg\n\nInfrarrojos Derecho\n\nInalámbrico Tx\n\nInalámbrico Rx\n\nSensor DTH Dato\n\nLibre\n\nCapacitivo 1\n\nCapacitivo 2\n\nCapacitivo 3\n\nCapacitivo 4\n\nI2C - SDA\n\nI2C - SCL\n\nLDR\n\nPotenciometro
 Wire Notes Line
 	800  1050 800  7000
@@
 NoConn ~ 5800 2700
 NoConn ~ 5800 2850
+NoConn ~ 7100 4800
 $EndSCHEMATC

Commit message: Revisado V0.4. Actualizados gerber y esquemas
Other:
- note added: "USB Tx\n\nUSB Rx\n\nEncoder canal A\n\nInterrupción Acelerómetro / Expansor GPIO\n\nReset Perifericos\n\nEncoder canal B\n\nInfrarrojos Izquierdo\n\nUltrasonidos Echo\n\nUltrasonidos Trigg\n\nInfrarrojos Derecho\n\nInalámbrico Tx\n\nInalámbrico Rx\n\nSensor DTH Dato\n\nLibre (Arduino LED)\n\nCapacitivo 1\n\nCapacitivo 2\n\nCapacitivo 3\n\nCapacitivo 4\n\nI2C - SDA\n\nI2C - SCL\n\nLDR\n\nPotenciom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"
- note removed: "USB Tx\n\nUSB Rx\n\nEncoder canal A\n\nInterrupción Acelerómetro\n\nReset Perifericos\n\nEncoder canal B\n\nInfrarrojos Izquierdo\n\nUltrasonidos Echo\n\nUltrasonidos Trigg\n\nInfrarrojos Derecho\n\nInalámbrico Tx\n\nInalámbrico Rx\n\nSensor DTH Dato\n\nLibre\n\nCapacitivo 1\n\nCapacitivo 2\n\nCapacitivo 3\n\nCapacitivo 4\n\nI2C - SDA\n\nI2C - SCL\n\nLDR\n\nPotenciometro"
Changed lines of the file:
@@
 Sheet 2 17
 Title "Control de la placa"
-Date "2017-01-19"
+Date "2017-01-25"
 Rev "V.0.4"
 Comp "NanoPlayBoard"
@@
 D0\n\nD1\n\nD2\n\nD3\n\nD4\n\nD5\n\nD6\n\nD7\n\nD8\n\nD9\n\nD10\n\nD11\n\nD12\n\nD13\n\nA0\n\nA1\n\nA2\n\nA3\n\nA4\n\nA5\n\nA6\n\nA7
 Text Notes 1250 6900 0    79   ~ 0
-USB Tx\n\nUSB Rx\n\nEncoder canal A\n\nInterrupción Acelerómetro\n\nReset Perifericos\n\nEncoder canal B\n\nInfrarrojos Izquierdo\n\nUltrasonidos Echo\n\nUltrasonidos Trigg\n\nInfrarrojos Derecho\n\nInalámbrico Tx\n\nInalámbrico Rx\n\nSensor DTH Dato\n\nLibre\n\nCapacitivo 1\n\nCapacitivo 2\n\nCapacitivo 3\n\nCapacitivo 4\n\nI2C - SDA\n\nI2C - SCL\n\nLDR\n\nPotenciometro
+USB Tx\n\nUSB Rx\n\nEncoder canal A\n\nInterrupción Acelerómetro / Expansor GPIO\n\nReset Perifericos\n\nEncoder canal B\n\nInfrarrojos Izquierdo\n\nUltrasonidos Echo\n\nUltrasonidos Trigg\n\nInfrarrojos Derecho\n\nInalámbrico Tx\n\nInalámbrico Rx\n\nSensor DTH Dato\n\nLibre (Arduino LED)\n\nCapacitivo 1\n\nCapacitivo 2\n\nCapacitivo 3\n\nCapacitivo 4\n\nI2C - SDA\n\nI2C - SCL\n\nLDR\n\nPotenciometro
 Wire Notes Line
 	800  1050 800  7000
