File: Acelerometro.sch (KiCad schematic (older format))
At the start: 9 parts, among them Q10 BSS138, Q9 BSS138, U7 MMA7660FC

Commit message: añaadido zocalo para sensor de temperatura y primera distribucion sobre la PCB
Parts:
- C5, C6: footprint Capacitors_ThroughHole:C_Disc_D3_P2.5 -> Capacitors_SMD:C_0805
- R31, R32, R33, R34: footprint (none) -> Resistors_SMD:R_0805
- U7: footprint (none) -> Housings_DFN_QFN:DFN-10-1EP_3x3mm_Pitch0.5mm
Changed lines of the file:
@@
 $Descr User 8268 5846
 encoding utf-8
-Sheet 13 13
+Sheet 13 14
 Title ""
 Date ""
@@
 	5200 1450 5200 1900
 $Comp
-L +3V3 #PWR044
+L +3V3 #PWR046
 U 1 1 57952AC0
 P 5200 1450
-F 0 "#PWR044" H 5200 1300 50  0001 C CNN
+F 0 "#PWR046" H 5200 1300 50  0001 C CNN
 F 1 "+3V3" H 5215 1623 50  0000 C CNN
 F 2 "" H 5200 1450 50  0000 C CNN
@@
 F 0 "R31" H 4220 1946 50  0000 L CNN
 F 1 "4K7" H 4220 1855 50  0000 L CNN
-F 2 "" V 4080 1900 50  0000 C CNN
+F 2 "Resistors_SMD:R_0805" V 4080 1900 50  0001 C CNN
 F 3 "" H 4150 1900 50  0000 C CNN
 F 4 "~" H 4150 1900 60  0001 C CNN "Fabricante"
@@
 	6200 1700 6200 1450
 $Comp
-L +5V #PWR045
+L +5V #PWR047
 U 1 1 57952EB0
 P 6200 1450
-F 0 "#PWR045" H 6200 1300 50  0001 C CNN
+F 0 "#PWR047" H 6200 1300 50  0001 C CNN
 F 1 "+5V" H 6215 1623 50  0000 C CNN
 F 2 "" H 6200 1450 50  0000 C CNN
@@
 	6500 1700 6500 1450
 $Comp
-L +5V #PWR046
+L +5V #PWR048
 U 1 1 57952EEB
 P 6500 1450
-F 0 "#PWR046" H 6500 1300 50  0001 C CNN
+F 0 "#PWR048" H 6500 1300 50  0001 C CNN
 F 1 "+5V" H 6515 1623 50  0000 C CNN
 F 2 "" H 6500 1450 50  0000 C CNN
@@
 F 0 "U7" H 2650 3077 100 0000 C CNN
 F 1 "MMA7660FC" H 2650 2911 100 0000 C CNN
-F 2 "" H 2500 2400 100 0001 C CNN
+F 2 "Housings_DFN_QFN:DFN-10-1EP_3x3mm_Pitch0.5mm" H 2500 2400 100 0001 C CNN
 F 3 "http://docs-europe.electrocomponents.com/webdocs/0ef4/0900766b80ef40cf.pdf" H 2500 2400 100 0001 C CNN
 F 4 "freescale" H 2650 2400 60  0001 C CNN "Fabricante"
@@
 	3550 2100 3550 3050
 $Comp
-L GND #PWR047
+L GND #PWR049
 U 1 1 579532CA
 P 3550 3050
-F 0 "#PWR047" H 3550 2800 50  0001 C CNN
+F 0 "#PWR049" H 3550 2800 50  0001 C CNN
 F 1 "GND" H 3555 2877 50  0000 C CNN
 F 2 "" H 3550 3050 50  0000 C CNN
@@
 	1750 2100 1750 3050
 $Comp
-L GND #PWR048
+L GND #PWR050
 U 1 1 5795333D
 P 1750 3050
-F 0 "#PWR048" H 1750 2800 50  0001 C CNN
+F 0 "#PWR050" H 1750 2800 50  0001 C CNN
 F 1 "GND" H 1755 2877 50  0000 C CNN
 F 2 "" H 1750 3050 50  0000 C CNN
@@
 	1900 2400 1900 1650
 $Comp
-L +3V3 #PWR049
+L +3V3 #PWR051
 U 1 1 579533C4
 P 1900 1650
-F 0 "#PWR049" H 1900 1500 50  0001 C CNN
+F 0 "#PWR051" H 1900 1500 50  0001 C CNN
 F 1 "+3V3" H 1915 1823 50  0000 C CNN
 F 2 "" H 1900 1650 50  0000 C CNN
@@
 	3400 2250 3400 1650
 $Comp
-L +3V3 #PWR050
+L +3V3 #PWR052
 U 1 1 57953474
 P 3400 1650
-F 0 "#PWR050" H 3400 1500 50  0001 C CNN
+F 0 "#PWR052" H 3400 1500 50  0001 C CNN
 F 1 "+3V3" H 3415 1823 50  0000 C CNN
 F 2 "" H 3400 1650 50  0000 C CNN
@@
 F 0 "R32" H 4570 1946 50  0000 L CNN
 F 1 "4K7" H 4570 1855 50  0000 L CNN
-F 2 "" V 4430 1900 50  0000 C CNN
+F 2 "Resistors_SMD:R_0805" V 4430 1900 50  0001 C CNN
 F 3 "" H 4500 1900 50  0000 C CNN
 F 4 "~" H 4500 1900 60  0001 C CNN "Fabricante"
@@
 F 0 "R33" H 6270 1896 50  0000 L CNN
 F 1 "4K7" H 6270 1805 50  0000 L CNN
-F 2 "" V 6130 1850 50  0000 C CNN
+F 2 "Resistors_SMD:R_0805" V 6130 1850 50  0001 C CNN
 F 3 "" H 6200 1850 50  0000 C CNN
 F 4 "~" H 6200 1850 60  0001 C CNN "Fabricante"
@@
 F 0 "R34" H 6570 1896 50  0000 L CNN
 F 1 "4K7" H 6570 1805 50  0000 L CNN
-F 2 "" V 6430 1850 50  0000 C CNN
+F 2 "Resistors_SMD:R_0805" V 6430 1850 50  0001 C CNN
 F 3 "" H 6500 1850 50  0000 C CNN
 F 4 "~" H 6500 1850 60  0001 C CNN "Fabricante"
@@
 F 0 "C5" H 2175 3750 50  0000 L CNN
 F 1 "100n" H 2175 3550 50  0000 L CNN
-F 2 "Capacitors_ThroughHole:C_Disc_D3_P2.5" H 2188 3500 50  0001 C CNN
+F 2 "Capacitors_SMD:C_0805" H 2188 3500 50  0001 C CNN
 F 3 "" H 2150 3650 50  0000 C CNN
 F 4 "~" H 2150 3650 60  0001 C CNN "Fabricante"
@@
 $EndComp
 $Comp
-L GND #PWR051
+L GND #PWR053
 U 1 1 57953EB4
 P 2150 3900
-F 0 "#PWR051" H 2150 3650 50  0001 C CNN
+F 0 "#PWR053" H 2150 3650 50  0001 C CNN
 F 1 "GND" H 2150 3750 50  0000 C CNN
 F 2 "" H 2150 3900 50  0000 C CNN
@@
 F 0 "C6" H 3125 3750 50  0000 L CNN
 F 1 "100n" H 3125 3550 50  0000 L CNN
-F 2 "Capacitors_ThroughHole:C_Disc_D3_P2.5" H 3138 3500 50  0001 C CNN
+F 2 "Capacitors_SMD:C_0805" H 3138 3500 50  0001 C CNN
 F 3 "" H 3100 3650 50  0000 C CNN
 F 4 "~" H 3100 3650 60  0001 C CNN "Fabricante"
@@
 $EndComp
 $Comp
-L GND #PWR052
+L GND #PWR054
 U 1 1 57953F7E
 P 3100 3900
-F 0 "#PWR052" H 3100 3650 50  0001 C CNN
+F 0 "#PWR054" H 3100 3650 50  0001 C CNN
 F 1 "GND" H 3100 3750 50  0000 C CNN
 F 2 "" H 3100 3900 50  0000 C CNN
@@
 	3100 3900 3100 3800
 $Comp
-L +3V3 #PWR053
+L +3V3 #PWR055
 U 1 1 57953FC4
 P 2150 3350
-F 0 "#PWR053" H 2150 3200 50  0001 C CNN
+F 0 "#PWR055" H 2150 3200 50  0001 C CNN
 F 1 "+3V3" H 2165 3523 50  0000 C CNN
 F 2 "" H 2150 3350 50  0000 C CNN
@@
 $EndComp
 $Comp
-L +3V3 #PWR054
+L +3V3 #PWR056
 U 1 1 57954005
 P 3100 3350
-F 0 "#PWR054" H 3100 3200 50  0001 C CNN
+F 0 "#PWR056" H 3100 3200 50  0001 C CNN
 F 1 "+3V3" H 3115 3523 50  0000 C CNN
 F 2 "" H 3100 3350 50  0000 C CNN

Commit message: ordenar referencias de componentes
Parts:
- C6: renamed from C5; Fabricante (none) -> SAMSUNG; Provedor (none) -> TME; Ref (none) -> CL21B104KBCNNNC; Ref_Proveedor (none) -> CL21B104KBCNNNC
- C7: renamed from C6; Fabricante (none) -> SAMSUNG; Provedor (none) -> TME; Ref (none) -> CL21B104KBCNNNC; Ref_Proveedor (none) -> CL21B104KBCNNNC
- R30: renamed from R31; Fabricante (none) -> VISHAY; Potencia (none) -> 1/8W; Provedor (none) -> TME; Ref (none) -> CRCW08054K70FKEA; Ref_Proveedor (none) -> CRCW08054K70FKEA; Tolerancia (none) -> 1%
- R31: renamed from R32; Fabricante (none) -> VISHAY; Potencia (none) -> 1/8W; Provedor (none) -> TME; Ref (none) -> CRCW08054K70FKEA; Ref_Proveedor (none) -> CRCW08054K70FKEA; Tolerancia (none) -> 1%
- R32: renamed from R33; Fabricante (none) -> VISHAY; Potencia (none) -> 1/8W; Provedor (none) -> TME; Ref (none) -> CRCW08054K70FKEA; Ref_Proveedor (none) -> CRCW08054K70FKEA; Tolerancia (none) -> 1%
- R33: renamed from R34; Fabricante (none) -> VISHAY; Potencia (none) -> 1/8W; Provedor (none) -> TME; Ref (none) -> CRCW08054K70FKEA; Ref_Proveedor (none) -> CRCW08054K70FKEA; Tolerancia (none) -> 1%
Changed lines of the file:
@@
 $Descr User 8268 5846
 encoding utf-8
-Sheet 13 15
+Sheet 12 15
 Title ""
 Date ""
@@
 	5200 1450 5200 1900
 $Comp
-L +3V3 #PWR039
+L +3V3 #PWR51
 U 1 1 57952AC0
 P 5200 1450
-F 0 "#PWR039" H 5200 1300 50  0001 C CNN
+F 0 "#PWR51" H 5200 1300 50  0001 C CNN
 F 1 "+3V3" H 5215 1623 50  0000 C CNN
 F 2 "" H 5200 1450 50  0000 C CNN
@@
 Connection ~ 5200 1600
 $Comp
-L R R31
+L R R30
 U 1 1 57952AE0
 P 4150 1900
-F 0 "R31" H 4220 1946 50  0000 L CNN
+F 0 "R30" H 4220 1946 50  0000 L CNN
 F 1 "4K7" H 4220 1855 50  0000 L CNN
 F 2 "Resistors_SMD:R_0805" V 4080 1900 50  0001 C CNN
 F 3 "" H 4150 1900 50  0000 C CNN
-F 4 "~" H 4150 1900 60  0001 C CNN "Fabricante"
-F 5 "~" H 4150 1900 60  0001 C CNN "Ref"
-F 6 "~" H 4150 1900 60  0001 C CNN "Potencia"
-F 7 "~" H 4150 1900 60  0001 C CNN "Tolerancia"
-F 8 "~" H 4150 1900 60  0001 C CNN "Provedor"
-F 9 "~" H 4150 1900 60  0001 C CNN "Ref_Proveedor"
+F 4 "VISHAY" H 1900 2300 60  0001 C CNN "Fabricante"
+F 5 "CRCW08054K70FKEA" H 1900 2300 60  0001 C CNN "Ref"
+F 6 "1/8W" H 1900 2300 60  0001 C CNN "Potencia"
+F 7 "1%" H 1900 2300 60  0001 C CNN "Tolerancia"
+F 8 "TME" H 1900 2300 60  0001 C CNN "Provedor"
+F 9 "CRCW08054K70FKEA" H 1900 2300 60  0001 C CNN "Ref_Proveedor"
 	1    4150 1900
 	1    0    0    -1
@@
 	6200 1700 6200 1450
 $Comp
-L +5V #PWR040
+L +5V #PWR52
 U 1 1 57952EB0
 P 6200 1450
-F 0 "#PWR040" H 6200 1300 50  0001 C CNN
+F 0 "#PWR52" H 6200 1300 50  0001 C CNN
 F 1 "+5V" H 6215 1623 50  0000 C CNN
 F 2 "" H 6200 1450 50  0000 C CNN
@@
 	6500 1700 6500 1450
 $Comp
-L +5V #PWR041
+L +5V #PWR53
 U 1 1 57952EEB
 P 6500 1450
-F 0 "#PWR041" H 6500 1300 50  0001 C CNN
+F 0 "#PWR53" H 6500 1300 50  0001 C CNN
 F 1 "+5V" H 6515 1623 50  0000 C CNN
 F 2 "" H 6500 1450 50  0000 C CNN
@@
 	3550 2100 3550 3050
 $Comp
-L GND #PWR042
+L GND #PWR50
 U 1 1 579532CA
 P 3550 3050
-F 0 "#PWR042" H 3550 2800 50  0001 C CNN
+F 0 "#PWR50" H 3550 2800 50  0001 C CNN
 F 1 "GND" H 3555 2877 50  0000 C CNN
 F 2 "" H 3550 3050 50  0000 C CNN
@@
 	1750 2100 1750 3050
 $Comp
-L GND #PWR043
+L GND #PWR43
 U 1 1 5795333D
 P 1750 3050
-F 0 "#PWR043" H 1750 2800 50  0001 C CNN
+F 0 "#PWR43" H 1750 2800 50  0001 C CNN
 F 1 "GND" H 1755 2877 50  0000 C CNN
 F 2 "" H 1750 3050 50  0000 C CNN
@@
 	1900 2400 1900 1650
 $Comp
-L +3V3 #PWR044
+L +3V3 #PWR44
 U 1 1 579533C4
 P 1900 1650
-F 0 "#PWR044" H 1900 1500 50  0001 C CNN
+F 0 "#PWR44" H 1900 1500 50  0001 C CNN
 F 1 "+3V3" H 1915 1823 50  0000 C CNN
 F 2 "" H 1900 1650 50  0000 C CNN
@@
 	3400 2250 3400 1650
 $Comp
-L +3V3 #PWR045
+L +3V3 #PWR49
 U 1 1 57953474
 P 3400 1650
-F 0 "#PWR045" H 3400 1500 50  0001 C CNN
+F 0 "#PWR49" H 3400 1500 50  0001 C CNN
 F 1 "+3V3" H 3415 1823 50  0000 C CNN
 F 2 "" H 3400 1650 50  0000 C CNN
@@
 NoConn ~ 2050 2700
 $Comp
-L R R32
+L R R31
 U 1 1 57953886
 P 4500 1900
-F 0 "R32" H 4570 1946 50  0000 L CNN
+F 0 "R31" H 4570 1946 50  0000 L CNN
 F 1 "4K7" H 4570 1855 50  0000 L CNN
 F 2 "Resistors_SMD:R_0805" V 4430 1900 50  0001 C CNN
 F 3 "" H 4500 1900 50  0000 C CNN
-F 4 "~" H 4500 1900 60  0001 C CNN "Fabricante"
-F 5 "~" H 4500 1900 60  0001 C CNN "Ref"
-F 6 "~" H 4500 1900 60  0001 C CNN "Potencia"
-F 7 "~" H 4500 1900 60  0001 C CNN "Tolerancia"
-F 8 "~" H 4500 1900 60  0001 C CNN "Provedor"
-F 9 "~" H 4500 1900 60  0001 C CNN "Ref_Proveedor"
+F 4 "VISHAY" H 1900 2300 60  0001 C CNN "Fabricante"
+F 5 "CRCW08054K70FKEA" H 1900 2300 60  0001 C CNN "Ref"
+F 6 "1/8W" H 1900 2300 60  0001 C CNN "Potencia"
+F 7 "1%" H 1900 2300 60  0001 C CNN "Tolerancia"
+F 8 "TME" H 1900 2300 60  0001 C CNN "Provedor"
+F 9 "CRCW08054K70FKEA" H 1900 2300 60  0001 C CNN "Ref_Proveedor"
 	1    4500 1900
 	1    0    0    -1
 $EndComp
 $Comp
-L R R33
+L R R32
 U 1 1 579538BB
 P 6200 1850
-F 0 "R33" H 6270 1896 50  0000 L CNN
+F 0 "R32" H 6270 1896 50  0000 L CNN
 F 1 "4K7" H 6270 1805 50  0000 L CNN
 F 2 "Resistors_SMD:R_0805" V 6130 1850 50  0001 C CNN
 F 3 "" H 6200 1850 50  0000 C CNN
-F 4 "~" H 6200 1850 60  0001 C CNN "Fabricante"
-F 5 "~" H 6200 1850 60  0001 C CNN "Ref"
-F 6 "~" H 6200 1850 60  0001 C CNN "Potencia"
-F 7 "~" H 6200 1850 60  0001 C CNN "Tolerancia"
-F 8 "~" H 6200 1850 60  0001 C CNN "Provedor"
-F 9 "~" H 6200 1850 60  0001 C CNN "Ref_Proveedor"
+F 4 "VISHAY" H 1900 2300 60  0001 C CNN "Fabricante"
+F 5 "CRCW08054K70FKEA" H 1900 2300 60  0001 C CNN "Ref"
+F 6 "1/8W" H 1900 2300 60  0001 C CNN "Potencia"
+F 7 "1%" H 1900 2300 60  0001 C CNN "Tolerancia"
+F 8 "TME" H 1900 2300 60  0001 C CNN "Provedor"
+F 9 "CRCW08054K70FKEA" H 1900 2300 60  0001 C CNN "Ref_Proveedor"
 	1    6200 1850
 	1    0    0    -1
 $EndComp
 $Comp
-L R R34
+L R R33
 U 1 1 57953937
 P 6500 1850
-F 0 "R34" H 6570 1896 50  0000 L CNN
+F 0 "R33" H 6570 1896 50  0000 L CNN
 F 1 "4K7" H 6570 1805 50  0000 L CNN
 F 2 "Resistors_SMD:R_0805" V 6430 1850 50  0001 C CNN
 F 3 "" H 6500 1850 50  0000 C CNN
-F 4 "~" H 6500 1850 60  0001 C CNN "Fabricante"
-F 5 "~" H 6500 1850 60  0001 C CNN "Ref"
-F 6 "~" H 6500 1850 60  0001 C CNN "Potencia"
-F 7 "~" H 6500 1850 60  0001 C CNN "Tolerancia"
-F 8 "~" H 6500 1850 60  0001 C CNN "Provedor"
-F 9 "~" H 6500 1850 60  0001 C CNN "Ref_Proveedor"
+F 4 "VISHAY" H 1900 2300 60  0001 C CNN "Fabricante"
+F 5 "CRCW08054K70FKEA" H 1900 2300 60  0001 C CNN "Ref"
+F 6 "1/8W" H 1900 2300 60  0001 C CNN "Potencia"
+F 7 "1%" H 1900 2300 60  0001 C CNN "Tolerancia"
+F 8 "TME" H 1900 2300 60  0001 C CNN "Provedor"
+F 9 "CRCW08054K70FKEA" H 1900 2300 60  0001 C CNN "Ref_Proveedor"
 	1    6500 1850
 	1    0    0    -1
 $EndComp
 $Comp
-L C C5
+L C C6
 U 1 1 57953EAD
 P 2150 3650
-F 0 "C5" H 2175 3750 50  0000 L CNN
+F 0 "C6" H 2175 3750 50  0000 L CNN
 F 1 "100n" H 2175 3550 50  0000 L CNN
 F 2 "Capacitors_SMD:C_0805" H 2188 3500 50  0001 C CNN
 F 3 "" H 2150 3650 50  0000 C CNN
-F 4 "~" H 2150 3650 60  0001 C CNN "Fabricante"
-F 5 "~" H 2150 3650 60  0001 C CNN "Ref"
-F 6 "~" H 2150 3650 60  0001 C CNN "Potencia"
-F 7 "~" H 2150 3650 60  0001 C CNN "Tolerancia"
-F 8 "~" H 2150 3650 60  0001 C CNN "Provedor"
-F 9 "~" H 2150 3650 60  0001 C CNN "Ref_Proveedor"
+F 4 "SAMSUNG" H 6450 1350 60  0001 C CNN "Fabricante"
+F 5 "CL21B104KBCNNNC" H 6450 1350 60  0001 C CNN "Ref"
+F 6 "~" H 6450 1350 60  0001 C CNN "Potencia"
+F 7 "~" H 6450 1350 60  0001 C CNN "Tolerancia"
+F 8 "TME" H 6450 1350 60  0001 C CNN "Provedor"
+F 9 "CL21B104KBCNNNC" H 6450 1350 60  0001 C CNN "Ref_Proveedor"
 	1    2150 3650
 	1    0    0    -1
 $EndComp
 $Comp
-L GND #PWR046
+L GND #PWR46
 U 1 1 57953EB4
 P 2150 3900
-F 0 "#PWR046" H 2150 3650 50  0001 C CNN
+F 0 "#PWR46" H 2150 3650 50  0001 C CNN
 F 1 "GND" H 2150 3750 50  0000 C CNN
 F 2 "" H 2150 3900 50  0000 C CNN
@@
 	2150 3900 2150 3800
 $Comp
-L C C6
+L C C7
 U 1 1 57953F77
 P 3100 3650
-F 0 "C6" H 3125 3750 50  0000 L CNN
+F 0 "C7" H 3125 3750 50  0000 L CNN
 F 1 "100n" H 3125 3550 50  0000 L CNN
 F 2 "Capacitors_SMD:C_0805" H 3138 3500 50  0001 C CNN
 F 3 "" H 3100 3650 50  0000 C CNN
-F 4 "~" H 3100 3650 60  0001 C CNN "Fabricante"
-F 5 "~" H 3100 3650 60  0001 C CNN "Ref"
-F 6 "~" H 3100 3650 60  0001 C CNN "Potencia"
-F 7 "~" H 3100 3650 60  0001 C CNN "Tolerancia"
-F 8 "~" H 3100 3650 60  0001 C CNN "Provedor"
-F 9 "~" H 3100 3650 60  0001 C CNN "Ref_Proveedor"
+F 4 "SAMSUNG" H 6450 1350 60  0001 C CNN "Fabricante"
+F 5 "CL21B104KBCNNNC" H 6450 1350 60  0001 C CNN "Ref"
+F 6 "~" H 6450 1350 60  0001 C CNN "Potencia"
+F 7 "~" H 6450 1350 60  0001 C CNN "Tolerancia"
+F 8 "TME" H 6450 1350 60  0001 C CNN "Provedor"
+F 9 "CL21B104KBCNNNC" H 6450 1350 60  0001 C CNN "Ref_Proveedor"
 	1    3100 3650
 	1    0    0    -1
 $EndComp
 $Comp
-L GND #PWR047
+L GND #PWR48
 U 1 1 57953F7E
 P 3100 3900
-F 0 "#PWR047" H 3100 3650 50  0001 C CNN
+F 0 "#PWR48" H 3100 3650 50  0001 C CNN
 F 1 "GND" H 3100 3750 50  0000 C CNN
 F 2 "" H 3100 3900 50  0000 C CNN
@@
 	3100 3900 3100 3800
 $Comp
-L +3V3 #PWR048
+L +3V3 #PWR45
 U 1 1 57953FC4
 P 2150 3350
-F 0 "#PWR048" H 2150 3200 50  0001 C CNN
+F 0 "#PWR45" H 2150 3200 50  0001 C CNN
 F 1 "+3V3" H 2165 3523 50  0000 C CNN
 F 2 "" H 2150 3350 50  0000 C CNN
@@
 $EndComp
 $Comp
-L +3V3 #PWR049
+L +3V3 #PWR47
 U 1 1 57954005
 P 3100 3350
-F 0 "#PWR049" H 3100 3200 50  0001 C CNN
+F 0 "#PWR47" H 3100 3200 50  0001 C CNN
 F 1 "+3V3" H 3115 3523 50  0000 C CNN
 F 2 "" H 3100 3350 50  0000 C CNN

Commit message: cambiados encoder y potenciometro
Parts:
- R30, R31, R32, R33: footprint Resistors_SMD:R_0805 -> Resistencias:R_0805
Changed lines of the file:
@@
 	5200 1450 5200 1900
 $Comp
-L +3V3 #PWR51
+L +3V3 #PWR045
 U 1 1 57952AC0
 P 5200 1450
-F 0 "#PWR51" H 5200 1300 50  0001 C CNN
+F 0 "#PWR045" H 5200 1300 50  0001 C CNN
 F 1 "+3V3" H 5215 1623 50  0000 C CNN
 F 2 "" H 5200 1450 50  0000 C CNN
@@
 F 0 "R30" H 4220 1946 50  0000 L CNN
 F 1 "4K7" H 4220 1855 50  0000 L CNN
-F 2 "Resistors_SMD:R_0805" V 4080 1900 50  0001 C CNN
+F 2 "Resistencias:R_0805" V 4080 1900 50  0001 C CNN
 F 3 "" H 4150 1900 50  0000 C CNN
 F 4 "VISHAY" H 1900 2300 60  0001 C CNN "Fabricante"
@@
 	6200 1700 6200 1450
 $Comp
-L +5V #PWR52
+L +5V #PWR046
 U 1 1 57952EB0
 P 6200 1450
-F 0 "#PWR52" H 6200 1300 50  0001 C CNN
+F 0 "#PWR046" H 6200 1300 50  0001 C CNN
 F 1 "+5V" H 6215 1623 50  0000 C CNN
 F 2 "" H 6200 1450 50  0000 C CNN
@@
 	6500 1700 6500 1450
 $Comp
-L +5V #PWR53
+L +5V #PWR047
 U 1 1 57952EEB
 P 6500 1450
-F 0 "#PWR53" H 6500 1300 50  0001 C CNN
+F 0 "#PWR047" H 6500 1300 50  0001 C CNN
 F 1 "+5V" H 6515 1623 50  0000 C CNN
 F 2 "" H 6500 1450 50  0000 C CNN
@@
 	3550 2100 3550 3050
 $Comp
-L GND #PWR50
+L GND #PWR048
 U 1 1 579532CA
 P 3550 3050
-F 0 "#PWR50" H 3550 2800 50  0001 C CNN
+F 0 "#PWR048" H 3550 2800 50  0001 C CNN
 F 1 "GND" H 3555 2877 50  0000 C CNN
 F 2 "" H 3550 3050 50  0000 C CNN
@@
 	1750 2100 1750 3050
 $Comp
-L GND #PWR43
+L GND #PWR049
 U 1 1 5795333D
 P 1750 3050
-F 0 "#PWR43" H 1750 2800 50  0001 C CNN
+F 0 "#PWR049" H 1750 2800 50  0001 C CNN
 F 1 "GND" H 1755 2877 50  0000 C CNN
 F 2 "" H 1750 3050 50  0000 C CNN
@@
 	1900 2400 1900 1650
 $Comp
-L +3V3 #PWR44
+L +3V3 #PWR050
 U 1 1 579533C4
 P 1900 1650
-F 0 "#PWR44" H 1900 1500 50  0001 C CNN
+F 0 "#PWR050" H 1900 1500 50  0001 C CNN
 F 1 "+3V3" H 1915 1823 50  0000 C CNN
 F 2 "" H 1900 1650 50  0000 C CNN
@@
 	3400 2250 3400 1650
 $Comp
-L +3V3 #PWR49
+L +3V3 #PWR051
 U 1 1 57953474
 P 3400 1650
-F 0 "#PWR49" H 3400 1500 50  0001 C CNN
+F 0 "#PWR051" H 3400 1500 50  0001 C CNN
 F 1 "+3V3" H 3415 1823 50  0000 C CNN
 F 2 "" H 3400 1650 50  0000 C CNN
@@
 F 0 "R31" H 4570 1946 50  0000 L CNN
 F 1 "4K7" H 4570 1855 50  0000 L CNN
-F 2 "Resistors_SMD:R_0805" V 4430 1900 50  0001 C CNN
+F 2 "Resistencias:R_0805" V 4430 1900 50  0001 C CNN
 F 3 "" H 4500 1900 50  0000 C CNN
 F 4 "VISHAY" H 1900 2300 60  0001 C CNN "Fabricante"
@@
 F 0 "R32" H 6270 1896 50  0000 L CNN
 F 1 "4K7" H 6270 1805 50  0000 L CNN
-F 2 "Resistors_SMD:R_0805" V 6130 1850 50  0001 C CNN
+F 2 "Resistencias:R_0805" V 6130 1850 50  0001 C CNN
 F 3 "" H 6200 1850 50  0000 C CNN
 F 4 "VISHAY" H 1900 2300 60  0001 C CNN "Fabricante"
@@
 F 0 "R33" H 6570 1896 50  0000 L CNN
 F 1 "4K7" H 6570 1805 50  0000 L CNN
-F 2 "Resistors_SMD:R_0805" V 6430 1850 50  0001 C CNN
+F 2 "Resistencias:R_0805" V 6430 1850 50  0001 C CNN
 F 3 "" H 6500 1850 50  0000 C CNN
 F 4 "VISHAY" H 1900 2300 60  0001 C CNN "Fabricante"
@@
 $EndComp
 $Comp
-L GND #PWR46
+L GND #PWR052
 U 1 1 57953EB4
 P 2150 3900
-F 0 "#PWR46" H 2150 3650 50  0001 C CNN
+F 0 "#PWR052" H 2150 3650 50  0001 C CNN
 F 1 "GND" H 2150 3750 50  0000 C CNN
 F 2 "" H 2150 3900 50  0000 C CNN
@@
 $EndComp
 $Comp
-L GND #PWR48
+L GND #PWR053
 U 1 1 57953F7E
 P 3100 3900
-F 0 "#PWR48" H 3100 3650 50  0001 C CNN
+F 0 "#PWR053" H 3100 3650 50  0001 C CNN
 F 1 "GND" H 3100 3750 50  0000 C CNN
 F 2 "" H 3100 3900 50  0000 C CNN
@@
 	3100 3900 3100 3800
 $Comp
-L +3V3 #PWR45
+L +3V3 #PWR054
 U 1 1 57953FC4
 P 2150 3350
-F 0 "#PWR45" H 2150 3200 50  0001 C CNN
+F 0 "#PWR054" H 2150 3200 50  0001 C CNN
 F 1 "+3V3" H 2165 3523 50  0000 C CNN
 F 2 "" H 2150 3350 50  0000 C CNN
@@
 $EndComp
 $Comp
-L +3V3 #PWR47
+L +3V3 #PWR055
 U 1 1 57954005
 P 3100 3350
-F 0 "#PWR47" H 3100 3200 50  0001 C CNN
+F 0 "#PWR055" H 3100 3200 50  0001 C CNN
 F 1 "+3V3" H 3115 3523 50  0000 C CNN
 F 2 "" H 3100 3350 50  0000 C CNN
