File: Acelerometro.sch (KiCad schematic (older format))
At the start: 9 parts, among them Q10 BSS138, Q9 BSS138, U7 MMA7660FC

Commit message: añadidos driver para led y conectores para fotodiodos infrarrojos
Parts:
- renumbered C6 to C13, C7 to C14, Q9 to Q6, Q10 to Q7, R30 to R32, R31 to R33, R32 to R34, R33 to R35, U7 to U8
Connections:
- net D3: now reaches U8.5 (~INT)
- no-connect marks 1 -> 0
Changed lines of the file:
@@
 EESchema Schematic File Version 2
+LIBS:Interfaces
+LIBS:Nano_PB-rescue
 LIBS:Sensores
 LIBS:power
@@
 LIBS:valves
 LIBS:MyLibrary
+LIBS:matriz_led
 LIBS:Nano_PB-cache
-EELAYER 25 0
+EELAYER 26 0
 EELAYER END
 $Descr User 8268 5846
 encoding utf-8
-Sheet 12 15
+Sheet 12 16
 Title "Acelerometro 3 ejes"
-Date "2016-08-07"
-Rev "V.0.2"
+Date "2017-01-04"
+Rev "V.0.3"
 Comp "NanoPlayBoard"
 Comment1 "Creada por Antonio Morales"
@@
 $EndDescr
 $Comp
-L BSS138 Q9
+L BSS138 Q6
 U 1 1 57952913
 P 5250 2100
-F 0 "Q9" V 5486 2100 50  0000 C CNN
+F 0 "Q6" V 5486 2100 50  0000 C CNN
 F 1 "BSS138" V 5577 2100 50  0000 C CNN
 F 2 "TO_SOT_Packages_SMD:SOT-23" H 5450 2025 50  0001 L CIN
@@
 	5200 1450 5200 1900
 $Comp
-L +3V3 #PWR045
+L +3V3 #PWR066
 U 1 1 57952AC0
 P 5200 1450
-F 0 "#PWR045" H 5200 1300 50  0001 C CNN
+F 0 "#PWR066" H 5200 1300 50  0001 C CNN
 F 1 "+3V3" H 5215 1623 50  0000 C CNN
 F 2 "" H 5200 1450 50  0000 C CNN
@@
 Connection ~ 5200 1600
 $Comp
-L R R30
+L R R32
 U 1 1 57952AE0
 P 4150 1900
-F 0 "R30" H 4220 1946 50  0000 L CNN
+F 0 "R32" H 4220 1946 50  0000 L CNN
 F 1 "4K7" H 4220 1855 50  0000 L CNN
 F 2 "Resistencias:R_0805" V 4080 1900 50  0001 C CNN
@@
 A5
 $Comp
-L BSS138 Q10
+L BSS138 Q7
 U 1 1 57952D65
 P 5900 2600
-F 0 "Q10" V 6136 2600 50  0000 C CNN
+F 0 "Q7" V 6136 2600 50  0000 C CNN
 F 1 "BSS138" V 6227 2600 50  0000 C CNN
 F 2 "TO_SOT_Packages_SMD:SOT-23" H 6100 2525 50  0001 L CIN
@@
 	6200 1700 6200 1450
 $Comp
-L +5V #PWR046
+L +5V #PWR067
 U 1 1 57952EB0
 P 6200 1450
-F 0 "#PWR046" H 6200 1300 50  0001 C CNN
+F 0 "#PWR067" H 6200 1300 50  0001 C CNN
 F 1 "+5V" H 6215 1623 50  0000 C CNN
 F 2 "" H 6200 1450 50  0000 C CNN
@@
 	6500 1700 6500 1450
 $Comp
-L +5V #PWR047
+L +5V #PWR068
 U 1 1 57952EEB
 P 6500 1450
-F 0 "#PWR047" H 6500 1300 50  0001 C CNN
+F 0 "#PWR068" H 6500 1300 50  0001 C CNN
 F 1 "+5V" H 6515 1623 50  0000 C CNN
 F 2 "" H 6500 1450 50  0000 C CNN
@@
 $EndComp
 $Comp
-L MMA7660FC U7
+L MMA7660FC U8
 U 1 1 57953056
 P 2650 2400
-F 0 "U7" H 2650 3077 100 0000 C CNN
+F 0 "U8" H 2650 3077 100 0000 C CNN
 F 1 "MMA7660FC" H 2650 2911 100 0000 C CNN
 F 2 "Housings_DFN_QFN:DFN-10-1EP_3x3mm_Pitch0.5mm" H 2500 2400 100 0001 C CNN
@@
 	3250 2100 3550 2100
 Wire Wire Line
-	2050 2550 1750 2550
-Connection ~ 1750 2550
-Wire Wire Line
-	1750 2100 2050 2100
+	2050 2550 1500 2550
+Connection ~ 1500 2550
+Wire Wire Line
+	1500 2100 2050 2100
 Wire Wire Line
 	3250 2400 3550 2400
@@
 	3550 2100 3550 3050
 $Comp
-L GND #PWR048
+L GND #PWR069
 U 1 1 579532CA
 P 3550 3050
-F 0 "#PWR048" H 3550 2800 50  0001 C CNN
+F 0 "#PWR069" H 3550 2800 50  0001 C CNN
 F 1 "GND" H 3555 2877 50  0000 C CNN
 F 2 "" H 3550 3050 50  0000 C CNN
@@
 Connection ~ 3550 2400
 Wire Wire Line
-	1750 2100 1750 3050
+	1500 2100 1500 3050
 $Comp
-L GND #PWR049
+L GND #PWR070
 U 1 1 5795333D
-P 1750 3050
-F 0 "#PWR049" H 1750 2800 50  0001 C CNN
-F 1 "GND" H 1755 2877 50  0000 C CNN
-F 2 "" H 1750 3050 50  0000 C CNN
-F 3 "" H 1750 3050 50  0000 C CNN
-	1    1750 3050
+P 1500 3050
+F 0 "#PWR070" H 1500 2800 50  0001 C CNN
+F 1 "GND" H 1505 2877 50  0000 C CNN
+F 2 "" H 1500 3050 50  0000 C CNN
+F 3 "" H 1500 3050 50  0000 C CNN
+	1    1500 3050
 	1    0    0    -1
 $EndComp
@@
 	1900 2400 1900 1650
 $Comp
-L +3V3 #PWR050
+L +3V3 #PWR071
 U 1 1 579533C4
 P 1900 1650
-F 0 "#PWR050" H 1900 1500 50  0001 C CNN
+F 0 "#PWR071" H 1900 1500 50  0001 C CNN
 F 1 "+3V3" H 1915 1823 50  0000 C CNN
 F 2 "" H 1900 1650 50  0000 C CNN
@@
 	3400 2250 3400 1650
 $Comp
-L +3V3 #PWR051
+L +3V3 #PWR072
 U 1 1 57953474
 P 3400 1650
-F 0 "#PWR051" H 3400 1500 50  0001 C CNN
+F 0 "#PWR072" H 3400 1500 50  0001 C CNN
 F 1 "+3V3" H 3415 1823 50  0000 C CNN
 F 2 "" H 3400 1650 50  0000 C CNN
@@
 	3900 2550 3250 2550
 Connection ~ 4150 2200
-NoConn ~ 2050 2700
 $Comp
-L R R31
+L R R33
 U 1 1 57953886
 P 4500 1900
-F 0 "R31" H 4570 1946 50  0000 L CNN
+F 0 "R33" H 4570 1946 50  0000 L CNN
 F 1 "4K7" H 4570 1855 50  0000 L CNN
 F 2 "Resistencias:R_0805" V 4430 1900 50  0001 C CNN
@@
 $EndComp
 $Comp
-L R R32
+L R R34
 U 1 1 579538BB
 P 6200 1850
-F 0 "R32" H 6270 1896 50  0000 L CNN
+F 0 "R34" H 6270 1896 50  0000 L CNN
 F 1 "4K7" H 6270 1805 50  0000 L CNN
 F 2 "Resistencias:R_0805" V 6130 1850 50  0001 C CNN
@@
 $EndComp
 $Comp
-L R R33
+L R R35
 U 1 1 57953937
 P 6500 1850
-F 0 "R33" H 6570 1896 50  0000 L CNN
+F 0 "R35" H 6570 1896 50  0000 L CNN
 F 1 "4K7" H 6570 1805 50  0000 L CNN
 F 2 "Resistencias:R_0805" V 6430 1850 50  0001 C CNN
@@
 $EndComp
 $Comp
-L C C6
+L C C13
 U 1 1 57953EAD
 P 2150 3650
-F 0 "C6" H 2175 3750 50  0000 L CNN
+F 0 "C13" H 2175 3750 50  0000 L CNN
 F 1 "100n" H 2175 3550 50  0000 L CNN
 F 2 "Capacitors_SMD:C_0805" H 2188 3500 50  0001 C CNN
@@
 $EndComp
 $Comp
-L GND #PWR052
+L GND #PWR073
 U 1 1 57953EB4
 P 2150 3900
-F 0 "#PWR052" H 2150 3650 50  0001 C CNN
+F 0 "#PWR073" H 2150 3650 50  0001 C CNN
 F 1 "GND" H 2150 3750 50  0000 C CNN
 F 2 "" H 2150 3900 50  0000 C CNN
@@
 	2150 3900 2150 3800
 $Comp
-L C C7
+L C C14
 U 1 1 57953F77
 P 3100 3650
-F 0 "C7" H 3125 3750 50  0000 L CNN
+F 0 "C14" H 3125 3750 50  0000 L CNN
 F 1 "100n" H 3125 3550 50  0000 L CNN
 F 2 "Capacitors_SMD:C_0805" H 3138 3500 50  0001 C CNN
@@
 $EndComp
 $Comp
-L GND #PWR053
+L GND #PWR074
 U 1 1 57953F7E
 P 3100 3900
-F 0 "#PWR053" H 3100 3650 50  0001 C CNN
+F 0 "#PWR074" H 3100 3650 50  0001 C CNN
 F 1 "GND" H 3100 3750 50  0000 C CNN
 F 2 "" H 3100 3900 50  0000 C CNN
@@
 	3100 3900 3100 3800
 $Comp
-L +3V3 #PWR054
+L +3V3 #PWR075
 U 1 1 57953FC4
 P 2150 3350
-F 0 "#PWR054" H 2150 3200 50  0001 C CNN
+F 0 "#PWR075" H 2150 3200 50  0001 C CNN
 F 1 "+3V3" H 2165 3523 50  0000 C CNN
 F 2 "" H 2150 3350 50  0000 C CNN
@@
 $EndComp
 $Comp
-L +3V3 #PWR055
+L +3V3 #PWR076
 U 1 1 57954005
 P 3100 3350
-F 0 "#PWR055" H 3100 3200 50  0001 C CNN
+F 0 "#PWR076" H 3100 3200 50  0001 C CNN
 F 1 "+3V3" H 3115 3523 50  0000 C CNN
 F 2 "" H 3100 3350 50  0000 C CNN
@@
 50 17 92 01 51 92 64 0C CE 27 7B 4E 87 A3 FC C9 E9 39 BC D0 3B DC 1F CF E6 3C 60 30 83 10 3D 18
 F4 0B 89 52 73 00 8B 80 91 08 28 22 8F 6D AB AA BD D3 E7 C4 3E A7 59 B4 A9 94 4D 1C A1 84 52 AC
-9A 46 F6 7A E1 FF 00 F0 A4 0C 74 26 CB 7B D1 00 00 00 00 49 45 4E 44 AE 42 60 82 00
+9A 46 F6 7A E1 FF 00 F0 A4 0C 74 26 CB 7B D1 00 00 00 00 49 45 4E 44 AE 42 60 82
 EndData
 $EndBitmap
+Wire Wire Line
+	2050 2700 1900 2700
+Text GLabel 1900 2700 0    50   Input ~ 0
+D3
 $EndSCHEMATC
