File: Potenciometro.sch (KiCad schematic (older format))
At the start: 1 part

Commit message: ordenar referencias de componentes
Parts:
- RV1: Fabricante SR PASSIVES -> ALPS; Potencia (none) -> 0,05W; Provedor TME -> RS; Ref R9011-1-10K -> RK09D1130C3W; Ref_Proveedor R9011-1-10K -> 729-3656; Tolerancia (none) -> 20%
Changed lines of the file:
@@
 $Descr User 8268 5846
 encoding utf-8
-Sheet 8 15
+Sheet 10 15
 Title ""
 Date ""
@@
 F 2 "Potenciometros:POT_SR_PASIVES_R9011" H 1650 1800 50  0001 C CNN
 F 3 "" H 1650 1800 50  0000 C CNN
-F 4 "SR PASSIVES" H 1650 1800 60  0001 C CNN "Fabricante"
-F 5 "R9011-1-10K" H 1650 1800 60  0001 C CNN "Ref"
-F 6 "~" H 1650 1800 60  0001 C CNN "Potencia"
-F 7 "~" H 1650 1800 60  0001 C CNN "Tolerancia"
-F 8 "TME" H 1650 1800 60  0001 C CNN "Provedor"
-F 9 "R9011-1-10K" H 1650 1800 60  0001 C CNN "Ref_Proveedor"
+F 4 "ALPS" H 1650 1800 60  0001 C CNN "Fabricante"
+F 5 "RK09D1130C3W" H 1650 1800 60  0001 C CNN "Ref"
+F 6 "0,05W" H 1650 1800 60  0001 C CNN "Potencia"
+F 7 "20%" H 1650 1800 60  0001 C CNN "Tolerancia"
+F 8 "RS" H 1650 1800 60  0001 C CNN "Provedor"
+F 9 "729-3656" H 1650 1800 60  0001 C CNN "Ref_Proveedor"
 	1    1650 1800
 	0    1    1    0
 $EndComp
 $Comp
-L +5V #PWR015
+L +5V #PWR26
 U 1 1 5793F637
 P 1650 1450
-F 0 "#PWR015" H 1650 1300 50  0001 C CNN
+F 0 "#PWR26" H 1650 1300 50  0001 C CNN
 F 1 "+5V" H 1650 1590 50  0000 C CNN
 F 2 "" H 1650 1450 50  0000 C CNN
@@
 $EndComp
 $Comp
-L GND #PWR016
+L GND #PWR27
 U 1 1 5793F63D
 P 1650 2300
-F 0 "#PWR016" H 1650 2050 50  0001 C CNN
+F 0 "#PWR27" H 1650 2050 50  0001 C CNN
 F 1 "GND" H 1650 2150 50  0000 C CNN
 F 2 "" H 1650 2300 50  0000 C CNN

Commit message: cambiados encoder y potenciometro
Parts:
- RV1: footprint Potenciometros:POT_SR_PASIVES_R9011 -> Potenciometros:ALP_RK09K111; Ref RK09D1130C3W -> RK09K1110A0J; Ref_Proveedor 729-3656 -> 729-3622
Changed lines of the file:
@@
 F 0 "RV1" H 1650 1720 50  0000 C CNN
 F 1 "10K" H 1650 1800 50  0000 C CNN
-F 2 "Potenciometros:POT_SR_PASIVES_R9011" H 1650 1800 50  0001 C CNN
+F 2 "Potenciometros:ALP_RK09K111" H 1650 1800 50  0001 C CNN
 F 3 "" H 1650 1800 50  0000 C CNN
 F 4 "ALPS" H 1650 1800 60  0001 C CNN "Fabricante"
-F 5 "RK09D1130C3W" H 1650 1800 60  0001 C CNN "Ref"
+F 5 "RK09K1110A0J" H 1650 1800 60  0001 C CNN "Ref"
 F 6 "0,05W" H 1650 1800 60  0001 C CNN "Potencia"
 F 7 "20%" H 1650 1800 60  0001 C CNN "Tolerancia"
 F 8 "RS" H 1650 1800 60  0001 C CNN "Provedor"
-F 9 "729-3656" H 1650 1800 60  0001 C CNN "Ref_Proveedor"
+F 9 "729-3622" H 1650 1800 60  0001 C CNN "Ref_Proveedor"
 	1    1650 1800
 	0    1    1    0
 $EndComp
 $Comp
-L +5V #PWR26
+L +5V #PWR028
 U 1 1 5793F637
 P 1650 1450
-F 0 "#PWR26" H 1650 1300 50  0001 C CNN
+F 0 "#PWR028" H 1650 1300 50  0001 C CNN
 F 1 "+5V" H 1650 1590 50  0000 C CNN
 F 2 "" H 1650 1450 50  0000 C CNN
@@
 $EndComp
 $Comp
-L GND #PWR27
+L GND #PWR029
 U 1 1 5793F63D
 P 1650 2300
-F 0 "#PWR27" H 1650 2050 50  0001 C CNN
+F 0 "#PWR029" H 1650 2050 50  0001 C CNN
 F 1 "GND" H 1650 2150 50  0000 C CNN
 F 2 "" H 1650 2300 50  0000 C CNN

Commit message: añadidos driver para led y conectores para fotodiodos infrarrojos
Parts:
- RV1: symbol POT -> POT-RESCUE-Nano_PB
Other:
- moved on the sheet: RV1
