File: Buzzer.sch (KiCad schematic (older format))
At the start: 2 parts

Commit message: corregidos valores en esquema y simbolos corruptos
Parts:
- SP1: symbol SPEAKER -> Speaker
Changed lines of the file:
@@
 EESchema Schematic File Version 2
-LIBS:Interfaces
 LIBS:Nano_PB-rescue
+LIBS:Interfaces
 LIBS:Sensores
 LIBS:power
@@
 LIBS:matriz_led
 LIBS:Pasivos
+LIBS:Reles
 LIBS:Nano_PB-cache
 EELAYER 26 0
@@
 $EndDescr
 $Comp
-L SPEAKER SP1
+L Speaker SP1
 U 1 1 5793E03E
-P 3850 2300
-F 0 "SP1" H 3750 2550 50  0000 C CNN
-F 1 "BUZZER" H 3750 2050 50  0000 C CNN
-F 2 "Buzzer:LOUDITY_LD-BZPN-1705" H 3850 2300 50  0001 C CNN
-F 3 "" H 3850 2300 50  0000 C CNN
-F 4 "LOUDITY" H 3850 2300 60  0001 C CNN "Fabricante"
-F 5 "LD-BZPN-1705" H 3850 2300 60  0001 C CNN "Ref"
-F 6 "~" H 3850 2300 60  0001 C CNN "Potencia"
-F 7 "~" H 3850 2300 60  0001 C CNN "Tolerancia"
-F 8 "TME" H 3850 2300 60  0001 C CNN "Provedor"
-F 9 "LD-BZPN-1705" H 3850 2300 60  0001 C CNN "Ref_Proveedor"
-	1    3850 2300
+P 3750 2200
+AR Path="/5793E03E" Ref="SP1"  Part="1"
+AR Path="/5793DF2F/5793E03E" Ref="SP1"  Part="1"
+F 0 "SP1" H 3650 2450 50  0000 C CNN
+F 1 "BUZZER" H 3650 1950 50  0000 C CNN
+F 2 "Buzzer:LOUDITY_LD-BZPN-1705" H 3750 2200 50  0001 C CNN
+F 3 "" H 3750 2200 50  0000 C CNN
+F 4 "LOUDITY" H 3750 2200 60  0001 C CNN "Fabricante"
+F 5 "LD-BZPN-1705" H 3750 2200 60  0001 C CNN "Ref"
+F 6 "~" H 3750 2200 60  0001 C CNN "Potencia"
+F 7 "~" H 3750 2200 60  0001 C CNN "Tolerancia"
+F 8 "TME" H 3750 2200 60  0001 C CNN "Provedor"
+F 9 "LD-BZPN-1705" H 3750 2200 60  0001 C CNN "Ref_Proveedor"
+	1    3750 2200
 	1    0    0    -1
 $EndComp
 $Comp
-L GND #PWR079
+L GND #PWR071
 U 1 1 5793E045
 P 3350 3000
-F 0 "#PWR079" H 3350 2750 50  0001 C CNN
+F 0 "#PWR071" H 3350 2750 50  0001 C CNN
 F 1 "GND" H 3350 2850 50  0000 C CNN
 F 2 "" H 3350 3000 50  0000 C CNN
@@
 	3000 2200 3550 2200
 Wire Wire Line
-	3350 2400 3350 3000
+	3350 2300 3350 3000
 Wire Wire Line
-	3550 2400 3350 2400
+	3550 2300 3350 2300
 Text GLabel 3000 2200 0    60   Input ~ 0
 BUZZER
 $Bitmap
 Pos 7500 4400
-Scale 0,350000
+Scale 0,000000
 Data
 89 50 4E 47 0D 0A 1A 0A 00 00 00 0D 49 48 44 52 00 00 01 D5 00 00 01 ED 08 06 00 00 00 4F 90 E4
@@
 $EndBitmap
 $Comp
-L +5V #PWR080
+L +5V #PWR072
 U 1 1 586FF93B
 P 3250 1450
-F 0 "#PWR080" H 3250 1300 50  0001 C CNN
+F 0 "#PWR072" H 3250 1300 50  0001 C CNN
 F 1 "+5V" H 3265 1623 50  0000 C CNN
 F 2 "" H 3250 1450 50  0000 C CNN
