File: Infrarrojos.sch (KiCad schematic (older format))
At the start: 12 parts, among them P11 CONN_01X04, P12 CONN_01X04, U9 40106

Commit message: finalizado enrutado provisional
Parts:
- P11, P12: footprint Pin_Headers:Pin_Header_Straight_1x03_Pitch2.54mm -> Pin_Headers:Pin_Header_Angled_1x04_Pitch2.54mm
Connections:
- net D6: now also U9.8 (Out); no longer U9.2 (Out)
- net D9: now also U9.2 (Out); no longer U9.4 (Out)
- net at C18.1, P11.4 (P4), R44.1: now also U9.9 (In); no longer U9.1 (In)
- net at C20.1, P12.4 (P4), R46.1: now also U9.1 (In); no longer U9.3 (In)
Changed lines of the file:
@@
 $Comp
 L 40106 U9
-U 1 1 587119F2
+U 4 1 587119F2
 P 2750 2700
 F 0 "U9" H 2750 3065 50  0000 C CNN
@@
 F 2 "Housings_SOIC:SOIC-16_3.9x9.9mm_Pitch1.27mm" H 2750 2700 50  0001 C CNN
 F 3 "" H 2750 2700 50  0001 C CNN
-	1    2750 2700
+F 4 "~" H 2750 2700 60  0001 C CNN "Fabricante"
+F 5 "~" H 2750 2700 60  0001 C CNN "Ref"
+F 6 "~" H 2750 2700 60  0001 C CNN "Potencia"
+F 7 "~" H 2750 2700 60  0001 C CNN "Tolerancia"
+F 8 "~" H 2750 2700 60  0001 C CNN "Provedor"
+F 9 "~" H 2750 2700 60  0001 C CNN "Ref_Proveedor"
+	4    2750 2700
 	0    1    1    0
 $EndComp
@@
 $EndComp
 $Comp
-L GND #PWR086
+L GND #PWR085
 U 1 1 58714E93
 P 950 2550
-F 0 "#PWR086" H 950 2300 50  0001 C CNN
+F 0 "#PWR085" H 950 2300 50  0001 C CNN
 F 1 "GND" H 950 2400 50  0000 C CNN
 F 2 "" H 950 2550 50  0000 C CNN
@@
 $EndComp
 $Comp
-L +5V #PWR087
+L +5V #PWR086
 U 1 1 58714E99
 P 950 1600
-F 0 "#PWR087" H 950 1450 50  0001 C CNN
+F 0 "#PWR086" H 950 1450 50  0001 C CNN
 F 1 "+5V" H 950 1740 50  0000 C CNN
 F 2 "" H 950 1600 50  0000 C CNN
@@
 $EndComp
 $Comp
-L GND #PWR088
+L GND #PWR087
 U 1 1 58714FB1
 P 1400 2700
-F 0 "#PWR088" H 1400 2450 50  0001 C CNN
+F 0 "#PWR087" H 1400 2450 50  0001 C CNN
 F 1 "GND" H 1405 2527 50  0000 C CNN
 F 2 "" H 1400 2700 50  0000 C CNN
@@
 $EndComp
 $Comp
-L GND #PWR089
+L GND #PWR088
 U 1 1 58714FD2
 P 1850 2700
-F 0 "#PWR089" H 1850 2450 50  0001 C CNN
+F 0 "#PWR088" H 1850 2450 50  0001 C CNN
 F 1 "GND" H 1855 2527 50  0000 C CNN
 F 2 "" H 1850 2700 50  0000 C CNN
@@
 $EndComp
 $Comp
-L GND #PWR090
+L GND #PWR089
 U 1 1 58714FEC
 P 2250 2700
-F 0 "#PWR090" H 2250 2450 50  0001 C CNN
+F 0 "#PWR089" H 2250 2450 50  0001 C CNN
 F 1 "GND" H 2255 2527 50  0000 C CNN
 F 2 "" H 2250 2700 50  0000 C CNN
@@
 F 0 "P11" H 3228 1891 50  0000 L CNN
 F 1 "CONN_01X04" H 3228 1800 50  0000 L CNN
-F 2 "Pin_Headers:Pin_Header_Straight_1x03_Pitch2.54mm" H 3150 1850 50  0001 C CNN
+F 2 "Pin_Headers:Pin_Header_Angled_1x04_Pitch2.54mm" H 3150 1850 50  0001 C CNN
 F 3 "" H 3150 1850 50  0000 C CNN
 	1    3150 1850
@@
 $EndComp
 $Comp
-L +5V #PWR091
+L +5V #PWR090
 U 1 1 5871561E
 P 2300 1450
-F 0 "#PWR091" H 2300 1300 50  0001 C CNN
+F 0 "#PWR090" H 2300 1300 50  0001 C CNN
 F 1 "+5V" H 2315 1623 50  0000 C CNN
 F 2 "" H 2300 1450 50  0000 C CNN
@@
 $Comp
 L 40106 U9
-U 2 1 5871655E
+U 1 1 5871655E
 P 6300 2700
 F 0 "U9" H 6300 3065 50  0000 C CNN
@@
 F 2 "Housings_SOIC:SOIC-16_3.9x9.9mm_Pitch1.27mm" H 6300 2700 50  0001 C CNN
 F 3 "" H 6300 2700 50  0001 C CNN
-	2    6300 2700
+F 4 "~" H 6300 2700 60  0001 C CNN "Fabricante"
+F 5 "~" H 6300 2700 60  0001 C CNN "Ref"
+F 6 "~" H 6300 2700 60  0001 C CNN "Potencia"
+F 7 "~" H 6300 2700 60  0001 C CNN "Tolerancia"
+F 8 "~" H 6300 2700 60  0001 C CNN "Provedor"
+F 9 "~" H 6300 2700 60  0001 C CNN "Ref_Proveedor"
+	1    6300 2700
 	0    1    1    0
 $EndComp
@@
 $EndComp
 $Comp
-L GND #PWR092
+L GND #PWR091
 U 1 1 58716572
 P 4500 2550
-F 0 "#PWR092" H 4500 2300 50  0001 C CNN
+F 0 "#PWR091" H 4500 2300 50  0001 C CNN
 F 1 "GND" H 4500 2400 50  0000 C CNN
 F 2 "" H 4500 2550 50  0000 C CNN
@@
 $EndComp
 $Comp
-L +5V #PWR093
+L +5V #PWR092
 U 1 1 58716578
 P 4500 1600
-F 0 "#PWR093" H 4500 1450 50  0001 C CNN
+F 0 "#PWR092" H 4500 1450 50  0001 C CNN
 F 1 "+5V" H 4500 1740 50  0000 C CNN
 F 2 "" H 4500 1600 50  0000 C CNN
@@
 $EndComp
 $Comp
-L GND #PWR094
+L GND #PWR093
 U 1 1 58716595
 P 4950 2700
-F 0 "#PWR094" H 4950 2450 50  0001 C CNN
+F 0 "#PWR093" H 4950 2450 50  0001 C CNN
 F 1 "GND" H 4955 2527 50  0000 C CNN
 F 2 "" H 4950 2700 50  0000 C CNN
@@
 $EndComp
 $Comp
-L GND #PWR095
+L GND #PWR094
 U 1 1 5871659B
 P 5400 2700
-F 0 "#PWR095" H 5400 2450 50  0001 C CNN
+F 0 "#PWR094" H 5400 2450 50  0001 C CNN
 F 1 "GND" H 5405 2527 50  0000 C CNN
 F 2 "" H 5400 2700 50  0000 C CNN
@@
 $EndComp
 $Comp
-L GND #PWR096
+L GND #PWR095
 U 1 1 587165A1
 P 5800 2700
-F 0 "#PWR096" H 5800 2450 50  0001 C CNN
+F 0 "#PWR095" H 5800 2450 50  0001 C CNN
 F 1 "GND" H 5805 2527 50  0000 C CNN
 F 2 "" H 5800 2700 50  0000 C CNN
@@
 F 0 "P12" H 6778 1891 50  0000 L CNN
 F 1 "CONN_01X04" H 6778 1800 50  0000 L CNN
-F 2 "Pin_Headers:Pin_Header_Straight_1x03_Pitch2.54mm" H 6700 1850 50  0001 C CNN
+F 2 "Pin_Headers:Pin_Header_Angled_1x04_Pitch2.54mm" H 6700 1850 50  0001 C CNN
 F 3 "" H 6700 1850 50  0000 C CNN
 	1    6700 1850
@@
 $EndComp
 $Comp
-L +5V #PWR097
+L +5V #PWR096
 U 1 1 587165B1
 P 5850 1450
-F 0 "#PWR097" H 5850 1300 50  0001 C CNN
+F 0 "#PWR096" H 5850 1300 50  0001 C CNN
 F 1 "+5V" H 5865 1623 50  0000 C CNN
 F 2 "" H 5850 1450 50  0000 C CNN
@@
 $EndComp
 $Comp
-L GND #PWR098
+L GND #PWR097
 U 1 1 58718ECD
 P 1900 4650
-F 0 "#PWR098" H 1900 4400 50  0001 C CNN
+F 0 "#PWR097" H 1900 4400 50  0001 C CNN
 F 1 "GND" H 1900 4500 50  0000 C CNN
 F 2 "" H 1900 4650 50  0000 C CNN
@@
 $EndComp
 $Comp
-L +5V #PWR099
+L +5V #PWR098
 U 1 1 58718ED3
 P 1900 3700
-F 0 "#PWR099" H 1900 3550 50  0001 C CNN
+F 0 "#PWR098" H 1900 3550 50  0001 C CNN
 F 1 "+5V" H 1900 3840 50  0000 C CNN
 F 2 "" H 1900 3700 50  0000 C CNN

Commit message: corregidos valores en esquema y simbolos corruptos
Parts:
- C18, C20: Fabricante (none) -> SAMSUNG; Provedor (none) -> tme; Ref (none) -> CL21B103JBANNNC; Ref_Proveedor (none) -> CL21B103JBANNNC
- P11, P12: Fabricante (none) -> NINIGI; Provedor (none) -> tme; Ref (none) -> ZL211-40KG-S; Ref_Proveedor (none) -> ZL211-40KG-S
- R43, R45: Fabricante (none) -> YAGEO; Provedor (none) -> TME; Ref (none) -> RC0805FR-07220RL; Ref_Proveedor (none) -> RC0805FR-07220R
- R44, R46: Fabricante (none) -> VISHAY; Potencia (none) -> 1/8W; Provedor (none) -> TME; Ref (none) -> CRCW080547K0FKEA; Ref_Proveedor (none) -> CRCW080547K0FKEA; Tolerancia (none) -> 1%
- U9: footprint Housings_SOIC:SOIC-16_3.9x9.9mm_Pitch1.27mm -> Housings_SOIC:SOIC-14_3.9x8.7mm_Pitch1.27mm; Fabricante (none) -> NXP; Provedor (none) -> TME; Ref (none) -> HEF40106BT.653; Ref_Proveedor (none) -> HEF40106BT
Changed lines of the file:
@@
 EESchema Schematic File Version 2
-LIBS:Interfaces
 LIBS:Nano_PB-rescue
+LIBS:Interfaces
 LIBS:Sensores
 LIBS:power
@@
 LIBS:matriz_led
 LIBS:Pasivos
+LIBS:Reles
 LIBS:Nano_PB-cache
 EELAYER 26 0
@@
 F 0 "U9" H 2750 3065 50  0000 C CNN
 F 1 "40106" H 2750 2974 50  0000 C CNN
-F 2 "Housings_SOIC:SOIC-16_3.9x9.9mm_Pitch1.27mm" H 2750 2700 50  0001 C CNN
+F 2 "Housings_SOIC:SOIC-14_3.9x8.7mm_Pitch1.27mm" H 2750 2700 50  0001 C CNN
 F 3 "" H 2750 2700 50  0001 C CNN
-F 4 "~" H 2750 2700 60  0001 C CNN "Fabricante"
-F 5 "~" H 2750 2700 60  0001 C CNN "Ref"
-F 6 "~" H 2750 2700 60  0001 C CNN "Potencia"
-F 7 "~" H 2750 2700 60  0001 C CNN "Tolerancia"
-F 8 "~" H 2750 2700 60  0001 C CNN "Provedor"
-F 9 "~" H 2750 2700 60  0001 C CNN "Ref_Proveedor"
+F 4 "NXP" H 6300 2700 60  0001 C CNN "Fabricante"
+F 5 "HEF40106BT.653" H 6300 2700 60  0001 C CNN "Ref"
+F 6 "~" H 6300 2700 60  0001 C CNN "Potencia"
+F 7 "~" H 6300 2700 60  0001 C CNN "Tolerancia"
+F 8 "TME" H 6300 2700 60  0001 C CNN "Provedor"
+F 9 "HEF40106BT" H 6300 2700 60  0001 C CNN "Ref_Proveedor"
 	4    2750 2700
 	0    1    1    0
@@
 $EndComp
 $Comp
-L GND #PWR088
+L GND #PWR080
 U 1 1 58714E93
 P 950 2550
-F 0 "#PWR088" H 950 2300 50  0001 C CNN
+F 0 "#PWR080" H 950 2300 50  0001 C CNN
 F 1 "GND" H 950 2400 50  0000 C CNN
 F 2 "" H 950 2550 50  0000 C CNN
@@
 $EndComp
 $Comp
-L +5V #PWR089
+L +5V #PWR081
 U 1 1 58714E99
 P 950 1600
-F 0 "#PWR089" H 950 1450 50  0001 C CNN
+F 0 "#PWR081" H 950 1450 50  0001 C CNN
 F 1 "+5V" H 950 1740 50  0000 C CNN
 F 2 "" H 950 1600 50  0000 C CNN
@@
 F 2 "Resistencias:R_0805" V 1330 2400 50  0001 C CNN
 F 3 "" H 1400 2400 50  0000 C CNN
+F 4 "YAGEO" H 2750 2700 60  0001 C CNN "Fabricante"
+F 5 "RC0805FR-07220RL" H 2750 2700 60  0001 C CNN "Ref"
+F 6 "~" H 2750 2700 60  0001 C CNN "Potencia"
+F 7 "~" H 2750 2700 60  0001 C CNN "Tolerancia"
+F 8 "TME" H 2750 2700 60  0001 C CNN "Provedor"
+F 9 "RC0805FR-07220R" H 2750 2700 60  0001 C CNN "Ref_Proveedor"
 	1    1400 2400
 	1    0    0    -1
@@
 F 2 "Resistencias:R_0805" V 1780 2400 50  0001 C CNN
 F 3 "" H 1850 2400 50  0000 C CNN
-F 4 "~" H 1850 2400 60  0001 C CNN "Fabricante"
-F 5 "~" H 1850 2400 60  0001 C CNN "Ref"
-F 6 "~" H 1850 2400 60  0001 C CNN "Potencia"
-F 7 "~" H 1850 2400 60  0001 C CNN "Tolerancia"
-F 8 "~" H 1850 2400 60  0001 C CNN "Provedor"
-F 9 "~" H 1850 2400 60  0001 C CNN "Ref_Proveedor"
+F 4 "VISHAY" H 4350 1650 60  0001 C CNN "Fabricante"
+F 5 "CRCW080547K0FKEA" H 4350 1650 60  0001 C CNN "Ref"
+F 6 "1/8W" H 4350 1650 60  0001 C CNN "Potencia"
+F 7 "1%" H 4350 1650 60  0001 C CNN "Tolerancia"
+F 8 "TME" H 4350 1650 60  0001 C CNN "Provedor"
+F 9 "CRCW080547K0FKEA" H 4350 1650 60  0001 C CNN "Ref_Proveedor"
 	1    1850 2400
 	1    0    0    -1
@@
 F 2 "Capacitors_SMD:C_0805" H 2288 2250 50  0001 C CNN
 F 3 "" H 2250 2400 50  0000 C CNN
+F 4 "SAMSUNG" H 7750 2850 60  0001 C CNN "Fabricante"
+F 5 "CL21B103JBANNNC" H 7750 2850 60  0001 C CNN "Ref"
+F 6 "~" H 7750 2850 60  0001 C CNN "Potencia"
+F 7 "~" H 7750 2850 60  0001 C CNN "Tolerancia"
+F 8 "tme" H 7750 2850 60  0001 C CNN "Provedor"
+F 9 "CL21B103JBANNNC" H 7750 2850 60  0001 C CNN "Ref_Proveedor"
 	1    2250 2400
 	1    0    0    -1
 $EndComp
 $Comp
-L GND #PWR090
+L GND #PWR082
 U 1 1 58714FB1
 P 1400 2700
-F 0 "#PWR090" H 1400 2450 50  0001 C CNN
+F 0 "#PWR082" H 1400 2450 50  0001 C CNN
 F 1 "GND" H 1405 2527 50  0000 C CNN
 F 2 "" H 1400 2700 50  0000 C CNN
@@
 $EndComp
 $Comp
-L GND #PWR091
+L GND #PWR083
 U 1 1 58714FD2
 P 1850 2700
-F 0 "#PWR091" H 1850 2450 50  0001 C CNN
+F 0 "#PWR083" H 1850 2450 50  0001 C CNN
 F 1 "GND" H 1855 2527 50  0000 C CNN
 F 2 "" H 1850 2700 50  0000 C CNN
@@
 $EndComp
 $Comp
-L GND #PWR092
+L GND #PWR084
 U 1 1 58714FEC
 P 2250 2700
-F 0 "#PWR092" H 2250 2450 50  0001 C CNN
+F 0 "#PWR084" H 2250 2450 50  0001 C CNN
 F 1 "GND" H 2255 2527 50  0000 C CNN
 F 2 "" H 2250 2700 50  0000 C CNN
@@
 F 2 "Pin_Headers:Pin_Header_Angled_1x04_Pitch2.54mm" H 3150 1850 50  0001 C CNN
 F 3 "" H 3150 1850 50  0000 C CNN
+F 4 "NINIGI" H 7750 2850 60  0001 C CNN "Fabricante"
+F 5 "ZL211-40KG-S" H 7750 2850 60  0001 C CNN "Ref"
+F 6 "~" H 7750 2850 60  0001 C CNN "Potencia"
+F 7 "~" H 7750 2850 60  0001 C CNN "Tolerancia"
+F 8 "tme" H 7750 2850 60  0001 C CNN "Provedor"
+F 9 "ZL211-40KG-S" H 7750 2850 60  0001 C CNN "Ref_Proveedor"
 	1    3150 1850
 	1    0    0    -1
 $EndComp
 $Comp
-L +5V #PWR093
+L +5V #PWR085
 U 1 1 5871561E
 P 2300 1450
-F 0 "#PWR093" H 2300 1300 50  0001 C CNN
+F 0 "#PWR085" H 2300 1300 50  0001 C CNN
 F 1 "+5V" H 2315 1623 50  0000 C CNN
 F 2 "" H 2300 1450 50  0000 C CNN
@@
 F 0 "U9" H 6300 3065 50  0000 C CNN
 F 1 "40106" H 6300 2974 50  0000 C CNN
-F 2 "Housings_SOIC:SOIC-16_3.9x9.9mm_Pitch1.27mm" H 6300 2700 50  0001 C CNN
+F 2 "Housings_SOIC:SOIC-14_3.9x8.7mm_Pitch1.27mm" H 6300 2700 50  0001 C CNN
 F 3 "" H 6300 2700 50  0001 C CNN
-F 4 "~" H 6300 2700 60  0001 C CNN "Fabricante"
-F 5 "~" H 6300 2700 60  0001 C CNN "Ref"
+F 4 "NXP" H 6300 2700 60  0001 C CNN "Fabricante"
+F 5 "HEF40106BT.653" H 6300 2700 60  0001 C CNN "Ref"
 F 6 "~" H 6300 2700 60  0001 C CNN "Potencia"
 F 7 "~" H 6300 2700 60  0001 C CNN "Tolerancia"
-F 8 "~" H 6300 2700 60  0001 C CNN "Provedor"
-F 9 "~" H 6300 2700 60  0001 C CNN "Ref_Proveedor"
+F 8 "TME" H 6300 2700 60  0001 C CNN "Provedor"
+F 9 "HEF40106BT" H 6300 2700 60  0001 C CNN "Ref_Proveedor"
 	1    6300 2700
 	0    1    1    0
@@
 $EndComp
 $Comp
-L GND #PWR094
+L GND #PWR086
 U 1 1 58716572
 P 4500 2550
-F 0 "#PWR094" H 4500 2300 50  0001 C CNN
+F 0 "#PWR086" H 4500 2300 50  0001 C CNN
 F 1 "GND" H 4500 2400 50  0000 C CNN
 F 2 "" H 4500 2550 50  0000 C CNN
@@
 $EndComp
 $Comp
-L +5V #PWR095
+L +5V #PWR087
 U 1 1 58716578
 P 4500 1600
-F 0 "#PWR095" H 4500 1450 50  0001 C CNN
+F 0 "#PWR087" H 4500 1450 50  0001 C CNN
 F 1 "+5V" H 4500 1740 50  0000 C CNN
 F 2 "" H 4500 1600 50  0000 C CNN
@@
 F 2 "Resistencias:R_0805" V 4880 2400 50  0001 C CNN
 F 3 "" H 4950 2400 50  0000 C CNN
+F 4 "YAGEO" H 2750 2700 60  0001 C CNN "Fabricante"
+F 5 "RC0805FR-07220RL" H 2750 2700 60  0001 C CNN "Ref"
+F 6 "~" H 2750 2700 60  0001 C CNN "Potencia"
+F 7 "~" H 2750 2700 60  0001 C CNN "Tolerancia"
+F 8 "TME" H 2750 2700 60  0001 C CNN "Provedor"
+F 9 "RC0805FR-07220R" H 2750 2700 60  0001 C CNN "Ref_Proveedor"
 	1    4950 2400
 	1    0    0    -1
@@
 F 2 "Resistencias:R_0805" V 5330 2400 50  0001 C CNN
 F 3 "" H 5400 2400 50  0000 C CNN
+F 4 "VISHAY" H 4350 1650 60  0001 C CNN "Fabricante"
+F 5 "CRCW080547K0FKEA" H 4350 1650 60  0001 C CNN "Ref"
+F 6 "1/8W" H 4350 1650 60  0001 C CNN "Potencia"
+F 7 "1%" H 4350 1650 60  0001 C CNN "Tolerancia"
+F 8 "TME" H 4350 1650 60  0001 C CNN "Provedor"
+F 9 "CRCW080547K0FKEA" H 4350 1650 60  0001 C CNN "Ref_Proveedor"
 	1    5400 2400
 	1    0    0    -1
@@
 F 2 "Capacitors_SMD:C_0805" H 5838 2250 50  0001 C CNN
 F 3 "" H 5800 2400 50  0000 C CNN
+F 4 "SAMSUNG" H 7750 2850 60  0001 C CNN "Fabricante"
+F 5 "CL21B103JBANNNC" H 7750 2850 60  0001 C CNN "Ref"
+F 6 "~" H 7750 2850 60  0001 C CNN "Potencia"
+F 7 "~" H 7750 2850 60  0001 C CNN "Tolerancia"
+F 8 "tme" H 7750 2850 60  0001 C CNN "Provedor"
+F 9 "CL21B103JBANNNC" H 7750 2850 60  0001 C CNN "Ref_Proveedor"
 	1    5800 2400
 	1    0    0    -1
 $EndComp
 $Comp
-L GND #PWR096
+L GND #PWR088
 U 1 1 58716595
 P 4950 2700
-F 0 "#PWR096" H 4950 2450 50  0001 C CNN
+F 0 "#PWR088" H 4950 2450 50  0001 C CNN
 F 1 "GND" H 4955 2527 50  0000 C CNN
 F 2 "" H 4950 2700 50  0000 C CNN
@@
 $EndComp
 $Comp
-L GND #PWR097
+L GND #PWR089
 U 1 1 5871659B
 P 5400 2700
-F 0 "#PWR097" H 5400 2450 50  0001 C CNN
+F 0 "#PWR089" H 5400 2450 50  0001 C CNN
 F 1 "GND" H 5405 2527 50  0000 C CNN
 F 2 "" H 5400 2700 50  0000 C CNN
@@
 $EndComp
 $Comp
-L GND #PWR098
+L GND #PWR090
 U 1 1 587165A1
 P 5800 2700
-F 0 "#PWR098" H 5800 2450 50  0001 C CNN
+F 0 "#PWR090" H 5800 2450 50  0001 C CNN
 F 1 "GND" H 5805 2527 50  0000 C CNN
 F 2 "" H 5800 2700 50  0000 C CNN
@@
 F 2 "Pin_Headers:Pin_Header_Angled_1x04_Pitch2.54mm" H 6700 1850 50  0001 C CNN
 F 3 "" H 6700 1850 50  0000 C CNN
+F 4 "NINIGI" H 7750 2850 60  0001 C CNN "Fabricante"
+F 5 "ZL211-40KG-S" H 7750 2850 60  0001 C CNN "Ref"
+F 6 "~" H 7750 2850 60  0001 C CNN "Potencia"
+F 7 "~" H 7750 2850 60  0001 C CNN "Tolerancia"
+F 8 "tme" H 7750 2850 60  0001 C CNN "Provedor"
+F 9 "ZL211-40KG-S" H 7750 2850 60  0001 C CNN "Ref_Proveedor"
 	1    6700 1850
 	1    0    0    -1
 $EndComp
 $Comp
-L +5V #PWR099
+L +5V #PWR091
 U 1 1 587165B1
 P 5850 1450
-F 0 "#PWR099" H 5850 1300 50  0001 C CNN
+F 0 "#PWR091" H 5850 1300 50  0001 C CNN
 F 1 "+5V" H 5865 1623 50  0000 C CNN
 F 2 "" H 5850 1450 50  0000 C CNN
@@
 $EndComp
 $Comp
-L GND #PWR0100
+L GND #PWR092
 U 1 1 58718ECD
 P 1900 4650
-F 0 "#PWR0100" H 1900 4400 50  0001 C CNN
+F 0 "#PWR092" H 1900 4400 50  0001 C CNN
 F 1 "GND" H 1900 4500 50  0000 C CNN
 F 2 "" H 1900 4650 50  0000 C CNN
@@
 $EndComp
 $Comp
-L +5V #PWR0101
+L +5V #PWR093
 U 1 1 58718ED3
 P 1900 3700
-F 0 "#PWR0101" H 1900 3550 50  0001 C CNN
+F 0 "#PWR093" H 1900 3550 50  0001 C CNN
 F 1 "+5V" H 1900 3840 50  0000 C CNN
 F 2 "" H 1900 3700 50  0000 C CNN
@@
 $Bitmap
 Pos 7500 4400
-Scale 0,350000
+Scale 0,000000
 Data
 89 50 4E 47 0D 0A 1A 0A 00 00 00 0D 49 48 44 52 00 00 01 D5 00 00 01 ED 08 06 00 00 00 4F 90 E4
