File: Nano_PB.sch (KiCad schematic (older format))
At the start: 0 parts

Commit message: Actualizado el esquema electrico
Other:
- note added: "Este diseño es Software Libre; usted puede redistribuirlo y/o modificarlo bajo los términos\nde la "GNU General Public License" como lo publica la "FSF Free Software Foundation", o \n(a su elección) de cualquier versión posterior.\n\nEste diseño es distribuido con la esperanza de que le sea útil, pero SIN NINGUNA GARANTIA; \nincluso sin la garantía implícita por la VENTA o EJERCICIO DE ALGUN PROP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"

Commit message: añadidos driver para led y conectores para fotodiodos infrarrojos
Changed lines of the file:
@@
 EESchema Schematic File Version 2
+LIBS:Interfaces
+LIBS:Nano_PB-rescue
 LIBS:Sensores
 LIBS:power
@@
 LIBS:valves
 LIBS:MyLibrary
+LIBS:matriz_led
 LIBS:Nano_PB-cache
-EELAYER 25 0
+EELAYER 26 0
 EELAYER END
 $Descr A4 11693 8268
 encoding utf-8
-Sheet 1 15
+Sheet 1 16
 Title "Nano Play Board"
-Date "2016-08-07"
-Rev "V.0.2"
+Date "2017-01-04"
+Rev "V.0.3"
 Comp "NanoPlayBoard"
 Comment1 "Creada por Antonio Morales"
@@
 $EndSheet
 $Sheet
-S 5250 1200 1200 800
+S 4550 1200 1200 800
 U 57939A23
 F0 "Matriz Led" 60
@@
 $EndSheet
 $Sheet
-S 3350 1200 1200 800
+S 3050 1200 1200 800
 U 5794B6BE
 F0 "Bluetooth" 60
@@
 $EndSheet
 $Sheet
-S 7150 1200 1200 800
+S 6050 1200 1200 800
 U 5793F6CB
 F0 "Servo" 60
@@
 $EndSheet
 $Sheet
-S 9050 1200 1200 800
+S 7550 1200 1200 800
 U 5793D145
 F0 "Led_RGB" 60
@@
 $EndSheet
 $Sheet
-S 9050 2550 1200 800
+S 9050 1200 1200 800
 U 57993DAA
 F0 "dth11" 60
@@
 10 42 08 21 54 8F 30 A7 22 84 10 42 08 A1 7A 84 73 A9 10 42 08 21 84 50 3D C2 7A 2A 42 08 21 84
 10 AA 47 98 53 11 42 08 21 84 50 3D C2 7E 7F 84 10 42 08 21 54 8F FE 7F 0B 07 BA 83 B7 6B 1C F8
-00 00 00 00 49 45 4E 44 AE 42 60 82 00
+00 00 00 00 49 45 4E 44 AE 42 60 82
 EndData
 $EndBitmap
@@
 50 17 92 01 51 92 64 0C CE 27 7B 4E 87 A3 FC C9 E9 39 BC D0 3B DC 1F CF E6 3C 60 30 83 10 3D 18
 F4 0B 89 52 73 00 8B 80 91 08 28 22 8F 6D AB AA BD D3 E7 C4 3E A7 59 B4 A9 94 4D 1C A1 84 52 AC
-9A 46 F6 7A E1 FF 00 F0 A4 0C 74 26 CB 7B D1 00 00 00 00 49 45 4E 44 AE 42 60 82 00
+9A 46 F6 7A E1 FF 00 F0 A4 0C 74 26 CB 7B D1 00 00 00 00 49 45 4E 44 AE 42 60 82
 EndData
 $EndBitmap
+$Sheet
+S 9050 2550 1200 800
+U 5870CC54
+F0 "Infrarrojos" 50
+F1 "Infrarrojos.sch" 50
+$EndSheet
 $EndSCHEMATC

Commit message: Se añade un expansor GPIO al esquema y se elminan registros y codificador
Changed lines of the file:
@@
 LIBS:MyLibrary
 LIBS:matriz_led
+LIBS:Pasivos
 LIBS:Nano_PB-cache
 EELAYER 26 0
@@
 $Descr A4 11693 8268
 encoding utf-8
-Sheet 1 16
+Sheet 1 17
 Title "Nano Play Board"
-Date "2017-01-04"
-Rev "V.0.3"
+Date "2017-01-19"
+Rev "V.0.4"
 Comp "NanoPlayBoard"
 Comment1 "Creada por Antonio Morales"
@@
 $EndSheet
 $Sheet
+S 6050 5200 1200 800
+U 587FC15A
+F0 "ExpansorGPIO" 50
+F1 "ExpansorGPIO.sch" 50
+$EndSheet
+$Sheet
 S 4550 1200 1200 800
 U 57939A23
@@
 $EndSheet
 $Sheet
-S 7150 5200 1200 800
+S 7550 5200 1200 800
 U 5793F670
 F0 "Pulsadores" 60
@@
 $EndSheet
 $Sheet
-S 5250 5200 1200 800
+S 4550 5200 1200 800
 U 5794B93F
 F0 "Acelerometro" 60
@@
 $EndSheet
 $Sheet
-S 3350 5200 1200 800
+S 3050 5200 1200 800
 U 5793DF2F
 F0 "Buzzer" 60
@@
 F1 "Encoder.sch" 60
 $EndSheet
+$Sheet
+S 9050 2550 1200 800
+U 5870CC54
+F0 "Infrarrojos" 50
+F1 "Infrarrojos.sch" 50
+$EndSheet
 $Bitmap
 Pos 5900 3650
@@
 EndData
 $EndBitmap
-$Sheet
-S 9050 2550 1200 800
-U 5870CC54
-F0 "Infrarrojos" 50
-F1 "Infrarrojos.sch" 50
-$EndSheet
 $EndSCHEMATC
